File: 70W-Amplifier.sch (KiCad schematic (older format))
At the start: 30 parts, among them J1 RF_OUT, J2 RF_IN, J3 LPF_IN, J4 LPF_OUT, J5 13.8V Input, J6 PTT, K1 G5V-2, Q1 2N3906, Q2 IRF530, Q3 IRF530, T1 BN43-202 2T:1T, T2 FERRITE TUBE 1T:3T, U1 L7805

Commit message: gg
Parts:
- added R6: Varies According to Band, symbol Xenir:Resistor
Connections:
- net at C4.2, Q2.1 (G), T1.C2B: now also R6.2
- net at C5.1, Q3.1 (G), T1.C3A: now also R6.1
Changed lines of the file:
@@
 	1    0    0    -1
 $EndComp
-Text GLabel 6150 4350 2    50   Input ~ 0
+Text GLabel 6050 4250 1    50   Input ~ 0
 BIAS
-Wire Wire Line
-	6150 4350 6050 4350
 Connection ~ 6050 4350
 $Comp
@@
 	9300 4150 9150 4150
 Connection ~ 9150 4150
+Wire Wire Line
+	6050 4350 6050 4250
+$Comp
+L Xenir:Resistor R6
+U 1 1 61C90F87
+P 6400 4400
+F 0 "R6" V 6400 4246 28  0000 C CNN
+F 1 "Varies According to Band" H 6400 4303 28  0000 C CNN
+F 2 "" H 6400 4300 50  0001 C CNN
+F 3 "" H 6400 4300 50  0001 C CNN
+	1    6400 4400
+	0    -1   -1   0
+$EndComp
+Wire Wire Line
+	6400 3950 6400 4200
+Wire Wire Line
+	6400 4950 6400 4600
 $EndSCHEMATC

Commit message: added foot
Parts:
- C1, C2, C3, C4, C5: footprint (none) -> Xenir:Capacitor 1206
- EC1, EC2: footprint (none) -> Capacitor_SMD:CP_Elec_6.3x7.7
- J1, J2, J3, J4: footprint (none) -> Connector_Coaxial:SMA_Amphenol_132289_EdgeMount
- J5, J6: footprint (none) -> Xenir:Power Connector
- JP1: footprint (none) -> Xenir:Jumper
- L1, T1, T2: footprint (none) -> Xenir:BN-43-202-Vertical
- Q2, Q3: footprint Package_TO_SOT_THT:TO-220-3_Vertical -> Xenir:TO-220-Horizontal
- R1, R2, R3, R4, R5, R6, R7: footprint (none) -> Xenir:Resistor 1206
- VR1: footprint (none) -> Xenir:Trimpot Vertical
Changed lines of the file:
@@
 F 0 "R1" H 4950 1996 28  0000 C CNN
 F 1 "10k" H 4950 2053 28  0000 C CNN
-F 2 "" H 4950 2050 50  0001 C CNN
+F 2 "Xenir:Resistor 1206" H 4950 2050 50  0001 C CNN
 F 3 "" H 4950 2050 50  0001 C CNN
 	1    4950 2150
@@
 F 0 "R2" V 5329 2382 28  0000 R CNN
 F 1 "10k" V 5272 2382 28  0000 R CNN
-F 2 "" H 5300 2350 50  0001 C CNN
+F 2 "Xenir:Resistor 1206" H 5300 2350 50  0001 C CNN
 F 3 "" H 5300 2350 50  0001 C CNN
 	1    5300 2450
@@
 F 0 "EC2" V 7071 1968 28  0000 L CNN
 F 1 "100uF" V 7128 1968 28  0000 L CNN
-F 2 "" H 7100 2000 50  0001 C CNN
+F 2 "Capacitor_SMD:CP_Elec_6.3x7.7" H 7100 2000 50  0001 C CNN
 F 3 "" H 7100 2000 50  0001 C CNN
 	1    7100 1950
@@
 F 0 "EC1" V 4271 1968 28  0000 L CNN
 F 1 "100uF" V 4328 1968 28  0000 L CNN
-F 2 "" H 4300 2000 50  0001 C CNN
+F 2 "Capacitor_SMD:CP_Elec_6.3x7.7" H 4300 2000 50  0001 C CNN
 F 3 "" H 4300 2000 50  0001 C CNN
 	1    4300 1950
@@
 F 0 "J5" H 3418 1475 50  0000 C CNN
 F 1 "13.8V Input" H 3418 1566 50  0000 C CNN
-F 2 "" H 3500 1800 50  0001 C CNN
+F 2 "Xenir:Power Connector" H 3500 1800 50  0001 C CNN
 F 3 "~" H 3500 1800 50  0001 C CNN
 	1    3500 1800
@@
 F 0 "J6" H 4868 2575 50  0000 C CNN
 F 1 "PTT" H 4868 2666 50  0000 C CNN
-F 2 "" H 4950 2900 50  0001 C CNN
+F 2 "Xenir:Power Connector" H 4950 2900 50  0001 C CNN
 F 3 "~" H 4950 2900 50  0001 C CNN
 	1    4950 2900
@@
 F 0 "VR1" H 8400 2100 50  0000 R CNN
 F 1 "1.5k" H 8500 1800 50  0000 R CNN
-F 2 "" H 8200 1950 50  0001 C CNN
+F 2 "Xenir:Trimpot Vertical" H 8200 1950 50  0001 C CNN
 F 3 "~" H 8200 1950 50  0001 C CNN
 	1    8200 1950
@@
 F 0 "R7" H 7400 1546 28  0000 C CNN
 F 1 "1k" H 7400 1603 28  0000 C CNN
-F 2 "" H 7400 1600 50  0001 C CNN
+F 2 "Xenir:Resistor 1206" H 7400 1600 50  0001 C CNN
 F 3 "" H 7400 1600 50  0001 C CNN
 	1    7400 1700
@@
 F 0 "C2" V 7671 2065 28  0000 L CNN
 F 1 ".1uF" V 7728 2065 28  0000 L CNN
-F 2 "" H 7700 1800 50  0001 C CNN
+F 2 "Xenir:Capacitor 1206" H 7700 1800 50  0001 C CNN
 F 3 "" H 7700 1800 50  0001 C CNN
 	1    7700 1950
@@
 F 0 "J2" H 2350 4450 50  0000 C CNN
 F 1 "RF_IN" H 2450 4550 50  0000 C CNN
-F 2 "" H 2200 4800 50  0001 C CNN
+F 2 "Connector_Coaxial:SMA_Amphenol_132289_EdgeMount" H 2200 4800 50  0001 C CNN
 F 3 "" H 2200 4800 50  0001 C CNN
 	1    2200 4650
@@
 F 0 "J1" H 2000 4050 50  0000 C CNN
 F 1 "RF_OUT" H 2050 4150 50  0000 C CNN
-F 2 "" H 1800 4400 50  0001 C CNN
+F 2 "Connector_Coaxial:SMA_Amphenol_132289_EdgeMount" H 1800 4400 50  0001 C CNN
 F 3 "" H 1800 4400 50  0001 C CNN
 	1    1800 4250
@@
 F 0 "T1" H 5000 3731 50  0000 C CNN
 F 1 "BN43-202 2T:1T" H 5000 3650 50  0000 C CNN
-F 2 "" H 5000 3750 50  0001 C CNN
+F 2 "Xenir:BN-43-202-Vertical" H 5000 3750 50  0001 C CNN
 F 3 "" H 5000 3750 50  0001 C CNN
 	1    5000 3750
@@
 F 0 "R3" V 5729 4482 28  0000 R CNN
 F 1 "10k" V 5672 4482 28  0000 R CNN
-F 2 "" H 5700 4450 50  0001 C CNN
+F 2 "Xenir:Resistor 1206" H 5700 4450 50  0001 C CNN
 F 3 "" H 5700 4450 50  0001 C CNN
 	1    5700 4550
@@
 F 0 "C3" V 6021 4615 28  0000 L CNN
 F 1 ".1uF" V 6078 4615 28  0000 L CNN
-F 2 "" H 6050 4350 50  0001 C CNN
+F 2 "Xenir:Capacitor 1206" H 6050 4350 50  0001 C CNN
 F 3 "" H 6050 4350 50  0001 C CNN
 	1    6050 4500
@@
 F 0 "Q2" H 7054 3996 50  0000 L CNN
 F 1 "IRF530" H 7054 3905 50  0000 L CNN
-F 2 "Package_TO_SOT_THT:TO-220-3_Vertical" H 7100 3875 50  0001 L CIN
+F 2 "Xenir:TO-220-Horizontal" H 7100 3875 50  0001 L CIN
 F 3 "http://www.irf.com/product-info/datasheets/data/irf540n.pdf" H 6850 3950 50  0001 L CNN
 	1    6850 3950
@@
 F 0 "Q3" H 7054 4904 50  0000 L CNN
 F 1 "IRF530" H 7054 4995 50  0000 L CNN
-F 2 "Package_TO_SOT_THT:TO-220-3_Vertical" H 7100 4875 50  0001 L CIN
+F 2 "Xenir:TO-220-Horizontal" H 7100 4875 50  0001 L CIN
 F 3 "http://www.irf.com/product-info/datasheets/data/irf540n.pdf" H 6850 4950 50  0001 L CNN
 	1    6850 4950
@@
 F 0 "R4" H 6750 3146 28  0000 C CNN
 F 1 "100" H 6750 3203 28  0000 C CNN
-F 2 "" H 6750 3200 50  0001 C CNN
+F 2 "Xenir:Resistor 1206" H 6750 3200 50  0001 C CNN
 F 3 "" H 6750 3200 50  0001 C CNN
 	1    6750 3300
@@
 F 0 "C4" V 6371 3715 28  0000 L CNN
 F 1 ".47uF" V 6428 3715 28  0000 L CNN
-F 2 "" H 6400 3450 50  0001 C CNN
+F 2 "Xenir:Capacitor 1206" H 6400 3450 50  0001 C CNN
 F 3 "" H 6400 3450 50  0001 C CNN
 	1    6400 3600
@@
 F 0 "C5" V 6371 5465 28  0000 L CNN
 F 1 ".47uF" V 6428 5465 28  0000 L CNN
-F 2 "" H 6400 5200 50  0001 C CNN
+F 2 "Xenir:Capacitor 1206" H 6400 5200 50  0001 C CNN
 F 3 "" H 6400 5200 50  0001 C CNN
 	1    6400 5350
@@
 F 0 "R5" H 6750 5546 28  0000 C CNN
 F 1 "100" H 6750 5603 28  0000 C CNN
-F 2 "" H 6750 5600 50  0001 C CNN
+F 2 "Xenir:Resistor 1206" H 6750 5600 50  0001 C CNN
 F 3 "" H 6750 5600 50  0001 C CNN
 	1    6750 5700
@@
 F 0 "T2" H 8250 4450 50  0000 C CNN
 F 1 "FERRITE TUBE 1T:3T" V 8350 4450 31  0000 C CNN
-F 2 "" H 8550 5150 50  0001 C CNN
+F 2 "Xenir:BN-43-202-Vertical" H 8550 5150 50  0001 C CNN
 F 3 "" H 8550 5150 50  0001 C CNN
 	1    8550 5150
@@
 F 0 "C1" V 7821 4615 28  0000 L CNN
 F 1 ".1uF" V 7878 4615 28  0000 L CNN
-F 2 "" H 7850 4350 50  0001 C CNN
+F 2 "Xenir:Capacitor 1206" H 7850 4350 50  0001 C CNN
 F 3 "" H 7850 4350 50  0001 C CNN
 	1    7850 4500
@@
 F 0 "L1" V 7750 3850 50  0000 L CNN
 F 1 "BN-43-202 2T" H 7700 4100 31  0000 L CNN
-F 2 "" H 7850 4100 50  0001 C CNN
+F 2 "Xenir:BN-43-202-Vertical" H 7850 4100 50  0001 C CNN
 F 3 "" H 7850 4100 50  0001 C CNN
 	1    7850 4000
@@
 F 0 "J3" V 9310 3680 50  0000 L CNN
 F 1 "LPF_IN" V 9401 3680 50  0000 L CNN
-F 2 "" H 9350 3750 50  0001 C CNN
+F 2 "Connector_Coaxial:SMA_Amphenol_132289_EdgeMount" H 9350 3750 50  0001 C CNN
 F 3 "" H 9350 3750 50  0001 C CNN
 	1    9350 3750
@@
 F 0 "J4" V 10160 3680 50  0000 L CNN
 F 1 "LPF_OUT" V 10251 3680 50  0000 L CNN
-F 2 "" H 10200 3750 50  0001 C CNN
+F 2 "Connector_Coaxial:SMA_Amphenol_132289_EdgeMount" H 10200 3750 50  0001 C CNN
 F 3 "" H 10200 3750 50  0001 C CNN
 	1    10200 3750
@@
 F 0 "JP1" H 9600 4300 50  0000 C CNN
 F 1 "LPF Bypass" H 9600 4050 50  0000 C CNN
-F 2 "" H 9600 4150 50  0001 C CNN
+F 2 "Xenir:Jumper" H 9600 4150 50  0001 C CNN
 F 3 "~" H 9600 4150 50  0001 C CNN
 	1    9600 4150
@@
 F 0 "R6" V 6400 4246 28  0000 C CNN
 F 1 "Varies According to Band" H 6400 4303 28  0000 C CNN
-F 2 "" H 6400 4300 50  0001 C CNN
+F 2 "Xenir:Resistor 1206" H 6400 4300 50  0001 C CNN
 F 3 "" H 6400 4300 50  0001 C CNN
 	1    6400 4400

Commit message: ddd
Parts:
- U1: footprint (none) -> Package_TO_SOT_SMD:SOT-223-3_TabPin2
Changed lines of the file:
@@
 F 0 "U1" H 6350 1942 50  0000 C CNN
 F 1 "L7805" H 6350 1851 50  0000 C CNN
-F 2 "" H 6375 1550 50  0001 L CIN
+F 2 "Package_TO_SOT_SMD:SOT-223-3_TabPin2" H 6375 1550 50  0001 L CIN
 F 3 "http://www.st.com/content/ccc/resource/technical/document/datasheet/41/4f/b3/b0/12/d4/47/88/CD00000444.pdf/files/CD00000444.pdf/jcr:content/translations/en.CD00000444.pdf" H 6350 1650 50  0001 C CNN
 	1    6350 1700

Commit message: still going
Parts:
- J1, J2: footprint Connector_Coaxial:SMA_Amphenol_132289_EdgeMount -> Xenir:BNC
- U1: footprint Package_TO_SOT_SMD:SOT-223-3_TabPin2 -> Package_TO_SOT_SMD:TO-252-3_TabPin2
Changed lines of the file:
@@
 F 0 "U1" H 6350 1942 50  0000 C CNN
 F 1 "L7805" H 6350 1851 50  0000 C CNN
-F 2 "Package_TO_SOT_SMD:SOT-223-3_TabPin2" H 6375 1550 50  0001 L CIN
+F 2 "Package_TO_SOT_SMD:TO-252-3_TabPin2" H 6375 1550 50  0001 L CIN
 F 3 "http://www.st.com/content/ccc/resource/technical/document/datasheet/41/4f/b3/b0/12/d4/47/88/CD00000444.pdf/files/CD00000444.pdf/jcr:content/translations/en.CD00000444.pdf" H 6350 1650 50  0001 C CNN
 	1    6350 1700
@@
 F 0 "J2" H 2350 4450 50  0000 C CNN
 F 1 "RF_IN" H 2450 4550 50  0000 C CNN
-F 2 "Connector_Coaxial:SMA_Amphenol_132289_EdgeMount" H 2200 4800 50  0001 C CNN
+F 2 "Xenir:BNC" H 2200 4800 50  0001 C CNN
 F 3 "" H 2200 4800 50  0001 C CNN
 	1    2200 4650
@@
 F 0 "J1" H 2000 4050 50  0000 C CNN
 F 1 "RF_OUT" H 2050 4150 50  0000 C CNN
-F 2 "Connector_Coaxial:SMA_Amphenol_132289_EdgeMount" H 1800 4400 50  0001 C CNN
+F 2 "Xenir:BNC" H 1800 4400 50  0001 C CNN
 F 3 "" H 1800 4400 50  0001 C CNN
 	1    1800 4250

Commit message: added splitter
Parts:
- removed J3: LPF_IN, Connector_Coaxial:SMA_Amphenol_132289_EdgeMount, symbol Xenir:PCB_SMA
- removed J4: LPF_OUT, Connector_Coaxial:SMA_Amphenol_132289_EdgeMount, symbol Xenir:PCB_SMA
- removed Q1: 2N3906, Package_TO_SOT_THT:TO-92_Inline, symbol Transistor_BJT:2N3906
- removed T1: BN43-202 2T:1T, Xenir:BN-43-202-Vertical, symbol Xenir:T50_SPLITTER
- removed T2: FERRITE TUBE 1T:3T, Xenir:BN-43-202-Vertical, symbol Xenir:T50_SPLITTER
- added J3: LPF_IN, Xenir:PCB-SMA-EDGE, symbol Xenir:PCB_SMA_EDGE
- added J4: LPF_OUT, Xenir:PCB-SMA-EDGE, symbol Xenir:PCB_SMA_EDGE
- added Q1: 2N3906-SMD, Package_TO_SOT_SMD:SOT-23, symbol Xenir:2N3906-SMD
- added T1: BN-43-202 1T:2T, Xenir:BN-43-202-Splitter-SMD, symbol Xenir:Splitter_Center_Tap
- added T2: Ferrite 1T:3T, Xenir:Ferrite-Tube-Splitter-SMD, symbol Xenir:Splitter_Center_Tap
Connections:
- net +12V: now also Q1.3 (C)
- net BIAS: now also T1.4
- net GND: now also J3.2, J4.2, T1.1, T2.1
- net LPF: now also J4.1
- net TRANSMIT_ON: now also Q1.2 (E)
- net at R1.1, R2.2: now also Q1.1 (B)
- net at K1.9: now also T1.2
- net at C5.1, Q3.1 (G), R6.1: now also T1.5
- net at C4.2, Q2.1 (G), R6.2: now also T1.3
- net at Q2.2 (D), R4.1: now also T2.5
- net at Q3.2 (D), R5.1: now also T2.3
- net at JP1.1: now also J3.1, T2.2
- net at C1.1, L1.2: now also T2.4
Changed lines of the file:
@@
-$EndComp
-$Comp
-L Transistor_BJT:2N3906 Q1
-U 1 1 61C4A74A
-P 5300 1800
-F 0 "Q1" V 5628 1800 50  0000 C CNN
-F 1 "2N3906" V 5537 1800 50  0000 C CNN
-F 2 "Package_TO_SOT_THT:TO-92_Inline" H 5500 1725 50  0001 L CIN
-F 3 "https://www.onsemi.com/pub/Collateral/2N3906-D.PDF" H 5300 1800 50  0001 L CNN
-	1    5300 1800
-	0    1    -1   0
 $EndComp
 $Comp
@@
 	2400 4650 3150 4650
 $Comp
-L Xenir:T50_SPLITTER T1
-U 1 1 61CB8C2A
-P 5000 3750
-F 0 "T1" H 5000 3731 50  0000 C CNN
-F 1 "BN43-202 2T:1T" H 5000 3650 50  0000 C CNN
-F 2 "Xenir:BN-43-202-Vertical" H 5000 3750 50  0001 C CNN
-F 3 "" H 5000 3750 50  0001 C CNN
-	1    5000 3750
-	1    0    0    -1
-$EndComp
-$Comp
 L power:GND #PWR07
 U 1 1 61CC3CE8
@@
 $EndComp
 Wire Wire Line
-	5350 4350 5350 4550
+	5350 4350 5350 4450
 $Comp
 L Xenir:Resistor R3
@@
 Wire Wire Line
 	5350 4350 5700 4350
-Connection ~ 5350 4350
 Connection ~ 5700 4350
 Wire Wire Line
@@
 Wire Wire Line
 	6400 5500 6400 5700
-$Comp
-L Xenir:T50_SPLITTER T2
-U 1 1 61CE7B62
-P 8550 5150
-F 0 "T2" H 8250 4450 50  0000 C CNN
-F 1 "FERRITE TUBE 1T:3T" V 8350 4450 31  0000 C CNN
-F 2 "Xenir:BN-43-202-Vertical" H 8550 5150 50  0001 C CNN
-F 3 "" H 8550 5150 50  0001 C CNN
-	1    8550 5150
-	-1   0    0    1
-$EndComp
 Wire Wire Line
 	6950 3300 8200 3300
-Wire Wire Line
-	8200 3300 8200 3950
 Connection ~ 6950 3300
-Wire Wire Line
-	8200 4950 8200 5700
 Wire Wire Line
 	8200 5700 6950 5700
 Connection ~ 6950 5700
 Wire Wire Line
-	8200 4350 8200 4550
+	8200 4350 8200 4450
 $Comp
 L Xenir:Capacitor C1
@@
 Wire Wire Line
 	8200 4350 7850 4350
-Connection ~ 8200 4350
 $Comp
 L power:+12V #PWR015
@@
 	1    8900 4750
 	1    0    0    -1
-$EndComp
-$Comp
-L Xenir:PCB_SMA J3
-U 1 1 61D30F44
-P 9350 3750
-F 0 "J3" V 9310 3680 50  0000 L CNN
-F 1 "LPF_IN" V 9401 3680 50  0000 L CNN
-F 2 "Connector_Coaxial:SMA_Amphenol_132289_EdgeMount" H 9350 3750 50  0001 C CNN
-F 3 "" H 9350 3750 50  0001 C CNN
-	1    9350 3750
-	0    1    1    0
-$EndComp
-$Comp
-L Xenir:PCB_SMA J4
-U 1 1 61D3410C
-P 10200 3750
-F 0 "J4" V 10160 3680 50  0000 L CNN
-F 1 "LPF_OUT" V 10251 3680 50  0000 L CNN
-F 2 "Connector_Coaxial:SMA_Amphenol_132289_EdgeMount" H 10200 3750 50  0001 C CNN
-F 3 "" H 10200 3750 50  0001 C CNN
-	1    10200 3750
-	0    1    1    0
 $EndComp
 $Comp
@@
 Wire Wire Line
 	6400 4950 6400 4600
+$Comp
+L Xenir:Splitter_Center_Tap T1
+U 1 1 61CE4121
+P 5000 3850
+F 0 "T1" H 5000 2600 50  0000 C CNN
+F 1 "BN-43-202 1T:2T" V 5250 3250 50  0000 C CNN
+F 2 "Xenir:BN-43-202-Splitter-SMD" H 5000 3850 50  0001 C CNN
+F 3 "" H 5000 3850 50  0001 C CNN
+	1    5000 3850
+	1    0    0    -1
+$EndComp
+Wire Wire Line
+	5350 3950 5350 4050
+Wire Wire Line
+	5350 4850 5350 4950
+$Comp
+L Xenir:2N3906-SMD Q1
+U 1 1 61CF1527
+P 5300 1800
+F 0 "Q1" H 5500 1875 50  0000 L CNN
+F 1 "2N3906-SMD" H 5500 1800 50  0000 L CNN
+F 2 "Package_TO_SOT_SMD:SOT-23" H 5500 1725 50  0001 L CIN
+F 3 "https://www.fairchildsemi.com/datasheets/2N/2N3906.pdf" H 5300 1800 50  0001 L CNN
+	1    5300 1800
+	0    -1   -1   0
+$EndComp
+$Comp
+L Xenir:PCB_SMA_EDGE J3
+U 1 1 61CF5952
+P 9350 3750
+F 0 "J3" H 9400 3650 50  0000 C CNN
+F 1 "LPF_IN" H 9350 3750 50  0000 C CNN
+F 2 "Xenir:PCB-SMA-EDGE" H 9350 3750 50  0001 C CNN
+F 3 "" H 9350 3750 50  0001 C CNN
+	1    9350 3750
+	0    1    1    0
+$EndComp
+$Comp
+L Xenir:PCB_SMA_EDGE J4
+U 1 1 61CF9C6B
+P 10200 3750
+F 0 "J4" H 10250 3650 50  0000 C CNN
+F 1 "LPF_OUT" H 10200 3750 50  0000 C CNN
+F 2 "Xenir:PCB-SMA-EDGE" H 10200 3750 50  0001 C CNN
+F 3 "" H 10200 3750 50  0001 C CNN
+	1    10200 3750
+	0    1    1    0
+$EndComp
+$Comp
+L Xenir:Splitter_Center_Tap T2
+U 1 1 61CFF29A
+P 8550 5050
+F 0 "T2" H 8550 3800 50  0000 C CNN
+F 1 "Ferrite 1T:3T" V 8800 4450 50  0000 C CNN
+F 2 "Xenir:Ferrite-Tube-Splitter-SMD" H 8550 5050 50  0001 C CNN
+F 3 "" H 8550 5050 50  0001 C CNN
+	1    8550 5050
+	-1   0    0    1
+$EndComp
+Wire Wire Line
+	8200 3300 8200 4050
+Wire Wire Line
+	8200 4850 8200 5700
 $EndSCHEMATC

Commit message: pcb work
Parts:
- J5: footprint Xenir:Power Connector -> Connector_BarrelJack:BarrelJack_Horizontal
- VR1: footprint Xenir:Trimpot Vertical -> Xenir:Trimpot_Horizontal
Changed lines of the file:
@@
 F 0 "J5" H 3418 1475 50  0000 C CNN
 F 1 "13.8V Input" H 3418 1566 50  0000 C CNN
-F 2 "Xenir:Power Connector" H 3500 1800 50  0001 C CNN
+F 2 "Connector_BarrelJack:BarrelJack_Horizontal" H 3500 1800 50  0001 C CNN
 F 3 "~" H 3500 1800 50  0001 C CNN
 	1    3500 1800
@@
 F 0 "VR1" H 8400 2100 50  0000 R CNN
 F 1 "1.5k" H 8500 1800 50  0000 R CNN
-F 2 "Xenir:Trimpot Vertical" H 8200 1950 50  0001 C CNN
+F 2 "Xenir:Trimpot_Horizontal" H 8200 1950 50  0001 C CNN
 F 3 "~" H 8200 1950 50  0001 C CNN
 	1    8200 1950

Commit message: added resistors
Parts:
- R4, R5, R6: footprint Xenir:Resistor 1206 -> Resistor_THT:R_Axial_DIN0414_L11.9mm_D4.5mm_P20.32mm_Horizontal
Connections:
- net GND: now also T1.2; no longer T1.1
- net at K1.9: now also T1.1; no longer T1.2
- net Q2Drain: now reaches Q2.2 (D), R4.1, T2.5
- net Q3Drain: now reaches Q3.2 (D), R5.1, T2.3
Changed lines of the file:
@@
 Wire Wire Line
 	2400 4650 3150 4650
-$Comp
-L power:GND #PWR07
-U 1 1 61CC3CE8
-P 4650 4150
-F 0 "#PWR07" H 4650 3900 50  0001 C CNN
-F 1 "GND" H 4655 3977 50  0000 C CNN
-F 2 "" H 4650 4150 50  0001 C CNN
-F 3 "" H 4650 4150 50  0001 C CNN
-	1    4650 4150
-	1    0    0    -1
-$EndComp
 Wire Wire Line
 	5350 4350 5350 4450
@@
 F 0 "R4" H 6750 3146 28  0000 C CNN
 F 1 "100" H 6750 3203 28  0000 C CNN
-F 2 "Xenir:Resistor 1206" H 6750 3200 50  0001 C CNN
+F 2 "Resistor_THT:R_Axial_DIN0414_L11.9mm_D4.5mm_P20.32mm_Horizontal" H 6750 3200 50  0001 C CNN
 F 3 "" H 6750 3200 50  0001 C CNN
 	1    6750 3300
@@
 F 0 "R5" H 6750 5546 28  0000 C CNN
 F 1 "100" H 6750 5603 28  0000 C CNN
-F 2 "Xenir:Resistor 1206" H 6750 5600 50  0001 C CNN
+F 2 "Resistor_THT:R_Axial_DIN0414_L11.9mm_D4.5mm_P20.32mm_Horizontal" H 6750 5600 50  0001 C CNN
 F 3 "" H 6750 5600 50  0001 C CNN
 	1    6750 5700
@@
 	1    0    0    -1
 $EndComp
-Wire Wire Line
-	3750 4750 4650 4750
 Text GLabel 3750 4350 2    50   Input ~ 0
 LPF
@@
 F 0 "R6" V 6400 4246 28  0000 C CNN
 F 1 "Varies According to Band" H 6400 4303 28  0000 C CNN
-F 2 "Xenir:Resistor 1206" H 6400 4300 50  0001 C CNN
+F 2 "Resistor_THT:R_Axial_DIN0414_L11.9mm_D4.5mm_P20.32mm_Horizontal" H 6400 4300 50  0001 C CNN
 F 3 "" H 6400 4300 50  0001 C CNN
 	1    6400 4400
@@
 Wire Wire Line
 	8200 4850 8200 5700
+Wire Wire Line
+	4650 4150 4200 4150
+Wire Wire Line
+	4200 4150 4200 4750
+Wire Wire Line
+	4200 4750 3750 4750
+$Comp
+L power:GND #PWR0101
+U 1 1 61E0D190
+P 4650 4750
+F 0 "#PWR0101" H 4650 4500 50  0001 C CNN
+F 1 "GND" H 4550 4750 50  0000 C CNN
+F 2 "" H 4650 4750 50  0001 C CNN
+F 3 "" H 4650 4750 50  0001 C CNN
+	1    4650 4750
+	1    0    0    -1
+$EndComp
+Text Label 6950 3650 0    50   ~ 0
+Q2Drain
+Text Label 6950 5350 0    50   ~ 0
+Q3Drain
 $EndSCHEMATC

Commit message: added source resistor/cap
Parts:
- added C6, C7: .2uF, Xenir:Capacitor 1206, symbol Xenir:Capacitor
- added R8, R9: .17, Resistor_SMD:R_2512_6332Metric, symbol Xenir:Resistor
Connections:
- net GND: now also C6.1, C7.1, R8.2, R9.2; no longer Q2.3 (S), Q3.3 (S)
- new net: C6.2, Q2.3 (S), R8.1
- new net: C7.2, Q3.3 (S), R9.1
Changed lines of the file:
@@
 U 1 1 61CD37AD
 P 6850 3950
-F 0 "Q2" H 7054 3996 50  0000 L CNN
-F 1 "IRF530" H 7054 3905 50  0000 L CNN
+F 0 "Q2" H 7000 4100 50  0000 L CNN
+F 1 "IRF530" H 6600 4100 50  0000 L CNN
 F 2 "Xenir:TO-220-Horizontal" H 7100 3875 50  0001 L CIN
 F 3 "http://www.irf.com/product-info/datasheets/data/irf540n.pdf" H 6850 3950 50  0001 L CNN
@@
 U 1 1 61CD4539
 P 6850 4950
-F 0 "Q3" H 7054 4904 50  0000 L CNN
-F 1 "IRF530" H 7054 4995 50  0000 L CNN
+F 0 "Q3" H 7000 5100 50  0000 L CNN
+F 1 "IRF530" H 6600 5100 50  0000 L CNN
 F 2 "Xenir:TO-220-Horizontal" H 7100 4875 50  0001 L CIN
 F 3 "http://www.irf.com/product-info/datasheets/data/irf540n.pdf" H 6850 4950 50  0001 L CNN
@@
 	1    0    0    1
 $EndComp
-Wire Wire Line
-	6950 4150 6950 4350
 $Comp
 L power:GND #PWR013
 U 1 1 61CD68E3
-P 7100 4400
-F 0 "#PWR013" H 7100 4150 50  0001 C CNN
-F 1 "GND" H 7105 4227 50  0000 C CNN
-F 2 "" H 7100 4400 50  0001 C CNN
-F 3 "" H 7100 4400 50  0001 C CNN
-	1    7100 4400
-	1    0    0    -1
-$EndComp
-Wire Wire Line
-	6950 4350 7100 4350
-Wire Wire Line
-	7100 4350 7100 4400
-Connection ~ 6950 4350
-Wire Wire Line
-	6950 4350 6950 4750
+P 7550 4500
+F 0 "#PWR013" H 7550 4250 50  0001 C CNN
+F 1 "GND" H 7555 4327 50  0000 C CNN
+F 2 "" H 7550 4500 50  0001 C CNN
+F 3 "" H 7550 4500 50  0001 C CNN
+	1    7550 4500
+	1    0    0    -1
+$EndComp
+Wire Wire Line
+	7550 4450 7550 4500
 Wire Wire Line
 	5350 3950 6400 3950
@@
 Text Label 6950 5350 0    50   ~ 0
 Q3Drain
+$Comp
+L Xenir:Resistor R8
+U 1 1 61E660AB
+P 7150 4150
+F 0 "R8" V 7200 4275 28  0000 R CNN
+F 1 ".17" V 7150 4275 28  0000 R CNN
+F 2 "Resistor_SMD:R_2512_6332Metric" H 7150 4050 50  0001 C CNN
+F 3 "" H 7150 4050 50  0001 C CNN
+	1    7150 4150
+	1    0    0    -1
+$EndComp
+$Comp
+L Xenir:Resistor R9
+U 1 1 61E6F0FA
+P 7150 4750
+F 0 "R9" V 7179 4682 28  0000 R CNN
+F 1 ".17" V 7122 4682 28  0000 R CNN
+F 2 "Resistor_SMD:R_2512_6332Metric" H 7150 4650 50  0001 C CNN
+F 3 "" H 7150 4650 50  0001 C CNN
+	1    7150 4750
+	1    0    0    -1
+$EndComp
+$Comp
+L Xenir:Capacitor C6
+U 1 1 61E6FCAB
+P 7100 4325
+F 0 "C6" V 7025 4250 28  0000 L CNN
+F 1 ".2uF" V 7200 4200 28  0000 L CNN
+F 2 "Xenir:Capacitor 1206" H 7100 4175 50  0001 C CNN
+F 3 "" H 7100 4175 50  0001 C CNN
+	1    7100 4325
+	-1   0    0    1
+$EndComp
+$Comp
+L Xenir:Capacitor C7
+U 1 1 61E706E7
+P 7100 4550
+F 0 "C7" V 7025 4475 28  0000 L CNN
+F 1 ".2uF" V 7200 4425 28  0000 L CNN
+F 2 "Xenir:Capacitor 1206" H 7100 4400 50  0001 C CNN
+F 3 "" H 7100 4400 50  0001 C CNN
+	1    7100 4550
+	-1   0    0    1
+$EndComp
+Wire Wire Line
+	6950 4550 6950 4750
+Connection ~ 6950 4750
+Wire Wire Line
+	6950 4325 6950 4150
+Connection ~ 6950 4150
+Wire Wire Line
+	7350 4150 7350 4325
+Wire Wire Line
+	7350 4450 7550 4450
+Wire Wire Line
+	7350 4750 7350 4550
+Connection ~ 7350 4450
+Wire Wire Line
+	7250 4325 7350 4325
+Connection ~ 7350 4325
+Wire Wire Line
+	7350 4325 7350 4450
+Wire Wire Line
+	7250 4550 7350 4550
+Connection ~ 7350 4550
+Wire Wire Line
+	7350 4550 7350 4450
 $EndSCHEMATC
