File: 70W-Amplifier.sch (KiCad schematic (older format))
At the start: 35 parts, among them J1 RF_OUT, J2 RF_IN, J3 LPF_IN, J4 LPF_OUT, J5 13.8V Input, J6 PTT, K1 G5V-2, Q1 2N3906-SMD, Q2 IRF530, Q3 IRF530, T1 BN-43-202 1T:2T, T2 Ferrite 1T:3T, U1 L7805

Commit message: changed to surface mount
Parts:
- K1: footprint Relay_THT:Relay_DPDT_Omron_G5V-2 -> Xenir:Relay_DPDT_Omron_G5V-2-SMD
- VR1: footprint Xenir:Trimpot_Horizontal -> Xenir:Trimpot_Horizontal_SMD
Changed lines of the file:
@@
 F 0 "VR1" H 8400 2100 50  0000 R CNN
 F 1 "1.5k" H 8500 1800 50  0000 R CNN
-F 2 "Xenir:Trimpot_Horizontal" H 8200 1950 50  0001 C CNN
+F 2 "Xenir:Trimpot_Horizontal_SMD" H 8200 1950 50  0001 C CNN
 F 3 "~" H 8200 1950 50  0001 C CNN
 	1    8200 1950
@@
 F 0 "K1" V 2683 4250 50  0000 C CNN
 F 1 "G5V-2" V 2774 4250 50  0000 C CNN
-F 2 "Relay_THT:Relay_DPDT_Omron_G5V-2" H 4100 4200 50  0001 L CNN
+F 2 "Xenir:Relay_DPDT_Omron_G5V-2-SMD" H 4100 4200 50  0001 L CNN
 F 3 "http://omronfs.omron.com/en_US/ecb/products/pdf/en-g5v_2.pdf" H 3450 4250 50  0001 C CNN
 	1    3450 4250

Commit message: finished
Parts:
- L1: footprint Xenir:BN-43-202-Vertical -> Xenir:BN-43-202-Vertical-SMD
- R4, R5, R6: footprint Resistor_THT:R_Axial_DIN0414_L11.9mm_D4.5mm_P20.32mm_Horizontal -> Xenir:LargeResistorSurfaceMount
Changed lines of the file:
@@
 F 0 "R4" H 6750 3146 28  0000 C CNN
 F 1 "100" H 6750 3203 28  0000 C CNN
-F 2 "Resistor_THT:R_Axial_DIN0414_L11.9mm_D4.5mm_P20.32mm_Horizontal" H 6750 3200 50  0001 C CNN
+F 2 "Xenir:LargeResistorSurfaceMount" H 6750 3200 50  0001 C CNN
 F 3 "" H 6750 3200 50  0001 C CNN
 	1    6750 3300
@@
 F 0 "R5" H 6750 5546 28  0000 C CNN
 F 1 "100" H 6750 5603 28  0000 C CNN
-F 2 "Resistor_THT:R_Axial_DIN0414_L11.9mm_D4.5mm_P20.32mm_Horizontal" H 6750 5600 50  0001 C CNN
+F 2 "Xenir:LargeResistorSurfaceMount" H 6750 5600 50  0001 C CNN
 F 3 "" H 6750 5600 50  0001 C CNN
 	1    6750 5700
@@
 F 0 "L1" V 7750 3850 50  0000 L CNN
 F 1 "BN-43-202 2T" H 7700 4100 31  0000 L CNN
-F 2 "Xenir:BN-43-202-Vertical" H 7850 4100 50  0001 C CNN
+F 2 "Xenir:BN-43-202-Vertical-SMD" H 7850 4100 50  0001 C CNN
 F 3 "" H 7850 4100 50  0001 C CNN
 	1    7850 4000
@@
 F 0 "R6" V 6400 4246 28  0000 C CNN
 F 1 "Varies According to Band" H 6400 4303 28  0000 C CNN
-F 2 "Resistor_THT:R_Axial_DIN0414_L11.9mm_D4.5mm_P20.32mm_Horizontal" H 6400 4300 50  0001 C CNN
+F 2 "Xenir:LargeResistorSurfaceMount" H 6400 4300 50  0001 C CNN
 F 3 "" H 6400 4300 50  0001 C CNN
 	1    6400 4400

Commit message: added gerber
Parts:
- J5: footprint Connector_BarrelJack:BarrelJack_Horizontal -> Xenir:PowerConnectorPads
- J6: footprint Xenir:Power Connector -> Xenir:TwoPads
Changed lines of the file:
@@
 F 0 "J5" H 3418 1475 50  0000 C CNN
 F 1 "13.8V Input" H 3418 1566 50  0000 C CNN
-F 2 "Connector_BarrelJack:BarrelJack_Horizontal" H 3500 1800 50  0001 C CNN
+F 2 "Xenir:PowerConnectorPads" H 3500 1800 50  0001 C CNN
 F 3 "~" H 3500 1800 50  0001 C CNN
 	1    3500 1800
@@
 F 0 "J6" H 4868 2575 50  0000 C CNN
 F 1 "PTT" H 4868 2666 50  0000 C CNN
-F 2 "Xenir:Power Connector" H 4950 2900 50  0001 C CNN
+F 2 "Xenir:TwoPads" H 4950 2900 50  0001 C CNN
 F 3 "~" H 4950 2900 50  0001 C CNN
 	1    4950 2900

Commit message: test
Other:
- note added: "Test"
Changed lines of the file:
@@
 Wire Wire Line
 	7350 4550 7350 4450
+Text Notes 3450 5600 0    50   ~ 0
+Test
 $EndSCHEMATC

Commit message: CHANGED BOARD SIZE
Other:
- note removed: "Test"
Changed lines of the file:
@@
 Wire Wire Line
 	7350 4550 7350 4450
-Text Notes 3450 5600 0    50   ~ 0
-Test
 $EndSCHEMATC

Commit message: fixed pnp wrong way around
Connections:
- net +12V: now also Q1.2 (E); no longer Q1.3 (C)
- net TRANSMIT_ON: now also Q1.3 (C); no longer Q1.2 (E)
Changed lines of the file:
@@
 F 3 "https://www.fairchildsemi.com/datasheets/2N/2N3906.pdf" H 5300 1800 50  0001 L CNN
 	1    5300 1800
-	0    -1   -1   0
+	0    1    -1   0
 $EndComp
 $Comp

Commit message: added dc block cap
Parts:
- added C8: .1uF, Xenir:Capacitor 1206, symbol Xenir:Capacitor
Connections:
- net at J3.1, JP1.1: now also C8.1; no longer T2.1
- new net: C8.2, T2.1
Other:
- moved on the sheet: J3, J4, JP1
Changed lines of the file:
@@
 L power:GND #PWR019
 U 1 1 61D35B7D
-P 9050 4450
-F 0 "#PWR019" H 9050 4200 50  0001 C CNN
-F 1 "GND" H 9055 4277 50  0000 C CNN
-F 2 "" H 9050 4450 50  0001 C CNN
-F 3 "" H 9050 4450 50  0001 C CNN
-	1    9050 4450
+P 9350 4450
+F 0 "#PWR019" H 9350 4200 50  0001 C CNN
+F 1 "GND" H 9355 4277 50  0000 C CNN
+F 2 "" H 9350 4450 50  0001 C CNN
+F 3 "" H 9350 4450 50  0001 C CNN
+	1    9350 4450
 	1    0    0    -1
 $EndComp
@@
 L power:GND #PWR020
 U 1 1 61D35F33
-P 9900 4450
-F 0 "#PWR020" H 9900 4200 50  0001 C CNN
-F 1 "GND" H 9905 4277 50  0000 C CNN
-F 2 "" H 9900 4450 50  0001 C CNN
-F 3 "" H 9900 4450 50  0001 C CNN
-	1    9900 4450
-	1    0    0    -1
-$EndComp
-Wire Wire Line
-	9150 4450 9150 4750
-Wire Wire Line
-	9150 4750 8900 4750
-Text GLabel 10200 4750 2    50   Input ~ 0
+P 10200 4450
+F 0 "#PWR020" H 10200 4200 50  0001 C CNN
+F 1 "GND" H 10205 4277 50  0000 C CNN
+F 2 "" H 10200 4450 50  0001 C CNN
+F 3 "" H 10200 4450 50  0001 C CNN
+	1    10200 4450
+	1    0    0    -1
+$EndComp
+Wire Wire Line
+	9450 4450 9450 4750
+Wire Wire Line
+	9450 4750 9200 4750
+Text GLabel 10500 4750 2    50   Input ~ 0
 LPF
 Wire Wire Line
-	10000 4450 10000 4750
-Wire Wire Line
-	10000 4750 10200 4750
+	10300 4450 10300 4750
+Wire Wire Line
+	10300 4750 10500 4750
 $Comp
 L Device:Jumper JP1
 U 1 1 61D3D93E
-P 9600 4750
-F 0 "JP1" H 9600 4900 50  0000 C CNN
-F 1 "LPF Bypass" H 9600 4650 50  0000 C CNN
-F 2 "Xenir:Jumper" H 9600 4750 50  0001 C CNN
-F 3 "~" H 9600 4750 50  0001 C CNN
-	1    9600 4750
-	1    0    0    -1
-$EndComp
-Wire Wire Line
-	9900 4750 10000 4750
-Connection ~ 10000 4750
-Wire Wire Line
-	9300 4750 9150 4750
-Connection ~ 9150 4750
+P 9900 4750
+F 0 "JP1" H 9900 4900 50  0000 C CNN
+F 1 "LPF Bypass" H 9900 4650 50  0000 C CNN
+F 2 "Xenir:Jumper" H 9900 4750 50  0001 C CNN
+F 3 "~" H 9900 4750 50  0001 C CNN
+	1    9900 4750
+	1    0    0    -1
+$EndComp
+Wire Wire Line
+	10200 4750 10300 4750
+Connection ~ 10300 4750
+Wire Wire Line
+	9600 4750 9450 4750
+Connection ~ 9450 4750
 Wire Wire Line
 	6050 4350 6050 4250
@@
 L Xenir:PCB_SMA_EDGE J3
 U 1 1 61CF5952
-P 9350 4350
-F 0 "J3" H 9400 4250 50  0000 C CNN
-F 1 "LPF_IN" H 9350 4350 50  0000 C CNN
-F 2 "Xenir:PCB-SMA-EDGE" H 9350 4350 50  0001 C CNN
-F 3 "" H 9350 4350 50  0001 C CNN
-	1    9350 4350
+P 9650 4350
+F 0 "J3" H 9700 4250 50  0000 C CNN
+F 1 "LPF_IN" H 9650 4350 50  0000 C CNN
+F 2 "Xenir:PCB-SMA-EDGE" H 9650 4350 50  0001 C CNN
+F 3 "" H 9650 4350 50  0001 C CNN
+	1    9650 4350
 	0    1    1    0
 $EndComp
@@
 L Xenir:PCB_SMA_EDGE J4
 U 1 1 61CF9C6B
-P 10200 4350
-F 0 "J4" H 10250 4250 50  0000 C CNN
-F 1 "LPF_OUT" H 10200 4350 50  0000 C CNN
-F 2 "Xenir:PCB-SMA-EDGE" H 10200 4350 50  0001 C CNN
-F 3 "" H 10200 4350 50  0001 C CNN
-	1    10200 4350
+P 10500 4350
+F 0 "J4" H 10550 4250 50  0000 C CNN
+F 1 "LPF_OUT" H 10500 4350 50  0000 C CNN
+F 2 "Xenir:PCB-SMA-EDGE" H 10500 4350 50  0001 C CNN
+F 3 "" H 10500 4350 50  0001 C CNN
+	1    10500 4350
 	0    1    1    0
 $EndComp
@@
 Wire Wire Line
 	7350 4550 7350 4450
+$Comp
+L Xenir:Capacitor C8
+U 1 1 61E9AE04
+P 9050 4750
+F 0 "C8" V 9021 4865 28  0000 L CNN
+F 1 ".1uF" V 9078 4865 28  0000 L CNN
+F 2 "Xenir:Capacitor 1206" H 9050 4600 50  0001 C CNN
+F 3 "" H 9050 4600 50  0001 C CNN
+	1    9050 4750
+	-1   0    0    1
+$EndComp
 $EndSCHEMATC

Commit message: added diode prot
Parts:
- added BIAS_IN1, BIAS_OUT1: Conn_01x01, Connector_PinHeader_1.00mm:PinHeader_1x01_P1.00mm_Vertical, symbol Connector_Generic:Conn_01x01
- added D2, D3, D4, D5, D6, D7: 1N914, Diode_SMD:D_SOD-323, symbol Diode:1N914
Connections:
- new net: D2.1 (K), D4.2 (A)
- new net: BIAS_IN1.1 (Pin_1), D2.2 (A)
- new net: D4.1 (K), D6.2 (A)
- new net: D6.1 (K), D7.2 (A)
- new net: D5.2 (A), D7.1 (K)
- new net: D3.2 (A), D5.1 (K)
- new net: BIAS_OUT1.1 (Pin_1), D3.1 (K)
Changed lines of the file:
@@
+	-1   0    0    1
+$EndComp
+$Comp
+L Diode:1N914 D2
+U 1 1 61E91B1A
+P 9250 2450
+F 0 "D2" H 9250 2233 50  0000 C CNN
+F 1 "1N914" H 9250 2324 50  0000 C CNN
+F 2 "Diode_SMD:D_SOD-323" H 9250 2275 50  0001 C CNN
+F 3 "http://www.vishay.com/docs/85622/1n914.pdf" H 9250 2450 50  0001 C CNN
+	1    9250 2450
+	-1   0    0    1
+$EndComp
+$Comp
+L Diode:1N914 D4
+U 1 1 61E92F86
+P 9550 2450
+F 0 "D4" H 9550 2233 50  0000 C CNN
+F 1 "1N914" H 9550 2324 50  0000 C CNN
+F 2 "Diode_SMD:D_SOD-323" H 9550 2275 50  0001 C CNN
+F 3 "http://www.vishay.com/docs/85622/1n914.pdf" H 9550 2450 50  0001 C CNN
+	1    9550 2450
+	-1   0    0    1
+$EndComp
+$Comp
+L Diode:1N914 D6
+U 1 1 61E93EBC
+P 9850 2450
+F 0 "D6" H 9850 2233 50  0000 C CNN
+F 1 "1N914" H 9850 2324 50  0000 C CNN
+F 2 "Diode_SMD:D_SOD-323" H 9850 2275 50  0001 C CNN
+F 3 "http://www.vishay.com/docs/85622/1n914.pdf" H 9850 2450 50  0001 C CNN
+	1    9850 2450
+	-1   0    0    1
+$EndComp
+$Comp
+L Diode:1N914 D7
+U 1 1 61E94F31
+P 9850 2750
+F 0 "D7" H 9850 2967 50  0000 C CNN
+F 1 "1N914" H 9850 2876 50  0000 C CNN
+F 2 "Diode_SMD:D_SOD-323" H 9850 2575 50  0001 C CNN
+F 3 "http://www.vishay.com/docs/85622/1n914.pdf" H 9850 2750 50  0001 C CNN
+	1    9850 2750
+	1    0    0    -1
+$EndComp
+$Comp
+L Diode:1N914 D5
+U 1 1 61E9657F
+P 9550 2750
+F 0 "D5" H 9550 2967 50  0000 C CNN
+F 1 "1N914" H 9550 2876 50  0000 C CNN
+F 2 "Diode_SMD:D_SOD-323" H 9550 2575 50  0001 C CNN
+F 3 "http://www.vishay.com/docs/85622/1n914.pdf" H 9550 2750 50  0001 C CNN
+	1    9550 2750
+	1    0    0    -1
+$EndComp
+$Comp
+L Diode:1N914 D3
+U 1 1 61E977BD
+P 9250 2750
+F 0 "D3" H 9250 2967 50  0000 C CNN
+F 1 "1N914" H 9250 2876 50  0000 C CNN
+F 2 "Diode_SMD:D_SOD-323" H 9250 2575 50  0001 C CNN
+F 3 "http://www.vishay.com/docs/85622/1n914.pdf" H 9250 2750 50  0001 C CNN
+	1    9250 2750
+	1    0    0    -1
+$EndComp
+Wire Wire Line
+	10000 2450 10000 2750
+$Comp
+L Connector_Generic:Conn_01x01 BIAS_IN1
+U 1 1 61EAA0AE
+P 8900 2450
+F 0 "BIAS_IN1" H 9000 2250 50  0000 C CNN
+F 1 "Conn_01x01" H 9000 2350 50  0000 C CNN
+F 2 "Connector_PinHeader_1.00mm:PinHeader_1x01_P1.00mm_Vertical" H 8900 2450 50  0001 C CNN
+F 3 "~" H 8900 2450 50  0001 C CNN
+	1    8900 2450
+	-1   0    0    1
+$EndComp
+$Comp
+L Connector_Generic:Conn_01x01 BIAS_OUT1
+U 1 1 61EAB06B
+P 8900 2750
+F 0 "BIAS_OUT1" H 9000 2850 50  0000 C CNN
+F 1 "Conn_01x01" H 9000 2950 50  0000 C CNN
+F 2 "Connector_PinHeader_1.00mm:PinHeader_1x01_P1.00mm_Vertical" H 8900 2750 50  0001 C CNN
+F 3 "~" H 8900 2750 50  0001 C CNN
+	1    8900 2750
 	-1   0    0    1
 $EndComp
