File: 70W-Amplifier.sch (KiCad schematic (older format))
At the start: 44 parts, among them J1 RF_OUT, J2 RF_IN, J3 LPF_IN, J4 LPF_OUT, J5 13.8V Input, J6 PTT, J7 Conn_01x02, J8 Conn_01x02, K1 G5V-2, Q1 2N3906-SMD, Q2 IRF530, Q3 IRF530, T1 BN-43-202 1T:2T, T2 Ferrite 1T:3T, U1 L7805

Commit message: gg
Parts:
- C1, C2, C3, C4, C5, C6, C7, C8: symbol 70W-Amplifier-rescue:Capacitor-Xenir-70W-Amplifier-rescue -> 70W-Amplifier-rescue:Capacitor-Xenir-70W-Amplifier-rescue-70W-Amplifier-rescue
- EC1, EC2: symbol 70W-Amplifier-rescue:Cap_Polarized-Xenir-70W-Amplifier-rescue -> 70W-Amplifier-rescue:Cap_Polarized-Xenir-70W-Amplifier-rescue-70W-Amplifier-rescue
- J1, J2: symbol 70W-Amplifier-rescue:BNC-Xenir-70W-Amplifier-rescue -> 70W-Amplifier-rescue:BNC-Xenir-70W-Amplifier-rescue-70W-Amplifier-rescue
- J3, J4: symbol 70W-Amplifier-rescue:PCB_SMA_EDGE-Xenir-70W-Amplifier-rescue -> 70W-Amplifier-rescue:PCB_SMA_EDGE-Xenir-70W-Amplifier-rescue-70W-Amplifier-rescue
- L1: symbol 70W-Amplifier-rescue:Inductor-Xenir-70W-Amplifier-rescue -> 70W-Amplifier-rescue:Inductor-Xenir-70W-Amplifier-rescue-70W-Amplifier-rescue
- Q1: symbol 70W-Amplifier-rescue:2N3906-SMD-Xenir-70W-Amplifier-rescue -> 70W-Amplifier-rescue:2N3906-SMD-Xenir-70W-Amplifier-rescue-70W-Amplifier-rescue
- R1, R2, R3, R4, R5, R6, R7, R8, R9: symbol 70W-Amplifier-rescue:Resistor-Xenir-70W-Amplifier-rescue -> 70W-Amplifier-rescue:Resistor-Xenir-70W-Amplifier-rescue-70W-Amplifier-rescue
- T1, T2: symbol 70W-Amplifier-rescue:Splitter_Center_Tap-Xenir-70W-Amplifier-rescue -> 70W-Amplifier-rescue:Splitter_Center_Tap-Xenir-70W-Amplifier-rescue-70W-Amplifier-rescue
Changed lines of the file:
@@
 $EndComp
 $Comp
-L 70W-Amplifier-rescue:Resistor-Xenir-70W-Amplifier-rescue R1
+L 70W-Amplifier-rescue:Resistor-Xenir-70W-Amplifier-rescue-70W-Amplifier-rescue R1
 U 1 1 61C4B77E
 P 4950 2150
@@
 $EndComp
 $Comp
-L 70W-Amplifier-rescue:Resistor-Xenir-70W-Amplifier-rescue R2
+L 70W-Amplifier-rescue:Resistor-Xenir-70W-Amplifier-rescue-70W-Amplifier-rescue R2
 U 1 1 61C4D74C
 P 5300 2450
@@
 	5300 2150 5300 2250
 $Comp
-L 70W-Amplifier-rescue:Cap_Polarized-Xenir-70W-Amplifier-rescue EC2
+L 70W-Amplifier-rescue:Cap_Polarized-Xenir-70W-Amplifier-rescue-70W-Amplifier-rescue EC2
 U 1 1 61C4EC77
 P 7100 1950
@@
 $EndComp
 $Comp
-L 70W-Amplifier-rescue:Cap_Polarized-Xenir-70W-Amplifier-rescue EC1
+L 70W-Amplifier-rescue:Cap_Polarized-Xenir-70W-Amplifier-rescue-70W-Amplifier-rescue EC1
 U 1 1 61C4FE0A
 P 4300 1950
@@
 $EndComp
 $Comp
-L 70W-Amplifier-rescue:Resistor-Xenir-70W-Amplifier-rescue R7
+L 70W-Amplifier-rescue:Resistor-Xenir-70W-Amplifier-rescue-70W-Amplifier-rescue R7
 U 1 1 61C5E001
 P 7400 1700
@@
 $EndComp
 $Comp
-L 70W-Amplifier-rescue:Capacitor-Xenir-70W-Amplifier-rescue C2
+L 70W-Amplifier-rescue:Capacitor-Xenir-70W-Amplifier-rescue-70W-Amplifier-rescue C2
 U 1 1 61C5E84F
 P 7700 1950
@@
 	8350 1950 8450 1950
 $Comp
-L 70W-Amplifier-rescue:BNC-Xenir-70W-Amplifier-rescue J2
+L 70W-Amplifier-rescue:BNC-Xenir-70W-Amplifier-rescue-70W-Amplifier-rescue J2
 U 1 1 61C68424
 P 2200 4650
@@
 $EndComp
 $Comp
-L 70W-Amplifier-rescue:BNC-Xenir-70W-Amplifier-rescue J1
+L 70W-Amplifier-rescue:BNC-Xenir-70W-Amplifier-rescue-70W-Amplifier-rescue J1
 U 1 1 61C69914
 P 1800 4250
@@
 	5350 4350 5350 4450
 $Comp
-L 70W-Amplifier-rescue:Resistor-Xenir-70W-Amplifier-rescue R3
+L 70W-Amplifier-rescue:Resistor-Xenir-70W-Amplifier-rescue-70W-Amplifier-rescue R3
 U 1 1 61CCDCF5
 P 5700 4550
@@
 $EndComp
 $Comp
-L 70W-Amplifier-rescue:Capacitor-Xenir-70W-Amplifier-rescue C3
+L 70W-Amplifier-rescue:Capacitor-Xenir-70W-Amplifier-rescue-70W-Amplifier-rescue C3
 U 1 1 61CCE86F
 P 6050 4500
@@
 	5350 4950 6400 4950
 $Comp
-L 70W-Amplifier-rescue:Resistor-Xenir-70W-Amplifier-rescue R4
+L 70W-Amplifier-rescue:Resistor-Xenir-70W-Amplifier-rescue-70W-Amplifier-rescue R4
 U 1 1 61CDA054
 P 6750 3300
@@
 $EndComp
 $Comp
-L 70W-Amplifier-rescue:Capacitor-Xenir-70W-Amplifier-rescue C4
+L 70W-Amplifier-rescue:Capacitor-Xenir-70W-Amplifier-rescue-70W-Amplifier-rescue C4
 U 1 1 61CDADD3
 P 6400 3600
@@
 	6400 3950 6650 3950
 $Comp
-L 70W-Amplifier-rescue:Capacitor-Xenir-70W-Amplifier-rescue C5
+L 70W-Amplifier-rescue:Capacitor-Xenir-70W-Amplifier-rescue-70W-Amplifier-rescue C5
 U 1 1 61CDF56C
 P 6400 5350
@@
 $EndComp
 $Comp
-L 70W-Amplifier-rescue:Resistor-Xenir-70W-Amplifier-rescue R5
+L 70W-Amplifier-rescue:Resistor-Xenir-70W-Amplifier-rescue-70W-Amplifier-rescue R5
 U 1 1 61CDFD89
 P 6750 5700
@@
 	8200 4350 8200 4450
 $Comp
-L 70W-Amplifier-rescue:Capacitor-Xenir-70W-Amplifier-rescue C1
+L 70W-Amplifier-rescue:Capacitor-Xenir-70W-Amplifier-rescue-70W-Amplifier-rescue C1
 U 1 1 61CECBAC
 P 7850 4500
@@
 LPF
 $Comp
-L 70W-Amplifier-rescue:Inductor-Xenir-70W-Amplifier-rescue L1
+L 70W-Amplifier-rescue:Inductor-Xenir-70W-Amplifier-rescue-70W-Amplifier-rescue L1
 U 1 1 61D26F6D
 P 7850 4000
@@
 	6050 4350 6050 4250
 $Comp
-L 70W-Amplifier-rescue:Resistor-Xenir-70W-Amplifier-rescue R6
+L 70W-Amplifier-rescue:Resistor-Xenir-70W-Amplifier-rescue-70W-Amplifier-rescue R6
 U 1 1 61C90F87
 P 6400 4400
@@
 	6400 4950 6400 4600
 $Comp
-L 70W-Amplifier-rescue:Splitter_Center_Tap-Xenir-70W-Amplifier-rescue T1
+L 70W-Amplifier-rescue:Splitter_Center_Tap-Xenir-70W-Amplifier-rescue-70W-Amplifier-rescue T1
 U 1 1 61CE4121
 P 5000 3850
@@
 	5350 4850 5350 4950
 $Comp
-L 70W-Amplifier-rescue:2N3906-SMD-Xenir-70W-Amplifier-rescue Q1
+L 70W-Amplifier-rescue:2N3906-SMD-Xenir-70W-Amplifier-rescue-70W-Amplifier-rescue Q1
 U 1 1 61CF1527
 P 5300 1800
@@
 $EndComp
 $Comp
-L 70W-Amplifier-rescue:PCB_SMA_EDGE-Xenir-70W-Amplifier-rescue J3
+L 70W-Amplifier-rescue:PCB_SMA_EDGE-Xenir-70W-Amplifier-rescue-70W-Amplifier-rescue J3
 U 1 1 61CF5952
 P 9650 4350
@@
 $EndComp
 $Comp
-L 70W-Amplifier-rescue:PCB_SMA_EDGE-Xenir-70W-Amplifier-rescue J4
+L 70W-Amplifier-rescue:PCB_SMA_EDGE-Xenir-70W-Amplifier-rescue-70W-Amplifier-rescue J4
 U 1 1 61CF9C6B
 P 10500 4350
@@
 $EndComp
 $Comp
-L 70W-Amplifier-rescue:Splitter_Center_Tap-Xenir-70W-Amplifier-rescue T2
+L 70W-Amplifier-rescue:Splitter_Center_Tap-Xenir-70W-Amplifier-rescue-70W-Amplifier-rescue T2
 U 1 1 61CFF29A
 P 8550 5050
@@
 Q3Drain
 $Comp
-L 70W-Amplifier-rescue:Resistor-Xenir-70W-Amplifier-rescue R8
+L 70W-Amplifier-rescue:Resistor-Xenir-70W-Amplifier-rescue-70W-Amplifier-rescue R8
 U 1 1 61E660AB
 P 7150 4150
@@
 $EndComp
 $Comp
-L 70W-Amplifier-rescue:Resistor-Xenir-70W-Amplifier-rescue R9
+L 70W-Amplifier-rescue:Resistor-Xenir-70W-Amplifier-rescue-70W-Amplifier-rescue R9
 U 1 1 61E6F0FA
 P 7150 4750
@@
 $EndComp
 $Comp
-L 70W-Amplifier-rescue:Capacitor-Xenir-70W-Amplifier-rescue C6
+L 70W-Amplifier-rescue:Capacitor-Xenir-70W-Amplifier-rescue-70W-Amplifier-rescue C6
 U 1 1 61E6FCAB
 P 7100 4325
@@
 $EndComp
 $Comp
-L 70W-Amplifier-rescue:Capacitor-Xenir-70W-Amplifier-rescue C7
+L 70W-Amplifier-rescue:Capacitor-Xenir-70W-Amplifier-rescue-70W-Amplifier-rescue C7
 U 1 1 61E706E7
 P 7100 4550
@@
 	7350 4550 7350 4450
 $Comp
-L 70W-Amplifier-rescue:Capacitor-Xenir-70W-Amplifier-rescue C8
+L 70W-Amplifier-rescue:Capacitor-Xenir-70W-Amplifier-rescue-70W-Amplifier-rescue C8
 U 1 1 61E9AE04
 P 9050 4750

Commit message: gg
Parts:
- C1, C2, C3, C4, C5, C6, C7, C8: symbol 70W-Amplifier-rescue:Capacitor-Xenir-70W-Amplifier-rescue-70W-Amplifier-rescue -> 70W-Amplifier-rescue:Capacitor-Xenir-70W-Amplifier-rescue-70W-Amplifier-rescue-70W-Amplifier-rescue
- EC1, EC2: symbol 70W-Amplifier-rescue:Cap_Polarized-Xenir-70W-Amplifier-rescue-70W-Amplifier-rescue -> 70W-Amplifier-rescue:Cap_Polarized-Xenir-70W-Amplifier-rescue-70W-Amplifier-rescue-70W-Amplifier-rescue
- J1, J2: symbol 70W-Amplifier-rescue:BNC-Xenir-70W-Amplifier-rescue-70W-Amplifier-rescue -> 70W-Amplifier-rescue:BNC-Xenir-70W-Amplifier-rescue-70W-Amplifier-rescue-70W-Amplifier-rescue
- J3, J4: symbol 70W-Amplifier-rescue:PCB_SMA_EDGE-Xenir-70W-Amplifier-rescue-70W-Amplifier-rescue -> 70W-Amplifier-rescue:PCB_SMA_EDGE-Xenir-70W-Amplifier-rescue-70W-Amplifier-rescue-70W-Amplifier-rescue
- L1: symbol 70W-Amplifier-rescue:Inductor-Xenir-70W-Amplifier-rescue-70W-Amplifier-rescue -> 70W-Amplifier-rescue:Inductor-Xenir-70W-Amplifier-rescue-70W-Amplifier-rescue-70W-Amplifier-rescue
- Q1: symbol 70W-Amplifier-rescue:2N3906-SMD-Xenir-70W-Amplifier-rescue-70W-Amplifier-rescue -> 70W-Amplifier-rescue:2N3906-SMD-Xenir-70W-Amplifier-rescue-70W-Amplifier-rescue-70W-Amplifier-rescue
- R1, R2, R3, R4, R5, R6, R7, R8, R9: symbol 70W-Amplifier-rescue:Resistor-Xenir-70W-Amplifier-rescue-70W-Amplifier-rescue -> 70W-Amplifier-rescue:Resistor-Xenir-70W-Amplifier-rescue-70W-Amplifier-rescue-70W-Amplifier-rescue
- T1, T2: symbol 70W-Amplifier-rescue:Splitter_Center_Tap-Xenir-70W-Amplifier-rescue-70W-Amplifier-rescue -> 70W-Amplifier-rescue:Splitter_Center_Tap-Xenir-70W-Amplifier-rescue-70W-Amplifier-rescue-70W-Amplifier-rescue
Changed lines of the file:
@@
 $EndComp
 $Comp
-L 70W-Amplifier-rescue:Resistor-Xenir-70W-Amplifier-rescue-70W-Amplifier-rescue R1
+L 70W-Amplifier-rescue:Resistor-Xenir-70W-Amplifier-rescue-70W-Amplifier-rescue-70W-Amplifier-rescue R1
 U 1 1 61C4B77E
 P 4950 2150
@@
 $EndComp
 $Comp
-L 70W-Amplifier-rescue:Resistor-Xenir-70W-Amplifier-rescue-70W-Amplifier-rescue R2
+L 70W-Amplifier-rescue:Resistor-Xenir-70W-Amplifier-rescue-70W-Amplifier-rescue-70W-Amplifier-rescue R2
 U 1 1 61C4D74C
 P 5300 2450
@@
 	5300 2150 5300 2250
 $Comp
-L 70W-Amplifier-rescue:Cap_Polarized-Xenir-70W-Amplifier-rescue-70W-Amplifier-rescue EC2
+L 70W-Amplifier-rescue:Cap_Polarized-Xenir-70W-Amplifier-rescue-70W-Amplifier-rescue-70W-Amplifier-rescue EC2
 U 1 1 61C4EC77
 P 7100 1950
@@
 $EndComp
 $Comp
-L 70W-Amplifier-rescue:Cap_Polarized-Xenir-70W-Amplifier-rescue-70W-Amplifier-rescue EC1
+L 70W-Amplifier-rescue:Cap_Polarized-Xenir-70W-Amplifier-rescue-70W-Amplifier-rescue-70W-Amplifier-rescue EC1
 U 1 1 61C4FE0A
 P 4300 1950
@@
 $EndComp
 $Comp
-L 70W-Amplifier-rescue:Resistor-Xenir-70W-Amplifier-rescue-70W-Amplifier-rescue R7
+L 70W-Amplifier-rescue:Resistor-Xenir-70W-Amplifier-rescue-70W-Amplifier-rescue-70W-Amplifier-rescue R7
 U 1 1 61C5E001
 P 7400 1700
@@
 $EndComp
 $Comp
-L 70W-Amplifier-rescue:Capacitor-Xenir-70W-Amplifier-rescue-70W-Amplifier-rescue C2
+L 70W-Amplifier-rescue:Capacitor-Xenir-70W-Amplifier-rescue-70W-Amplifier-rescue-70W-Amplifier-rescue C2
 U 1 1 61C5E84F
 P 7700 1950
@@
 	8350 1950 8450 1950
 $Comp
-L 70W-Amplifier-rescue:BNC-Xenir-70W-Amplifier-rescue-70W-Amplifier-rescue J2
+L 70W-Amplifier-rescue:BNC-Xenir-70W-Amplifier-rescue-70W-Amplifier-rescue-70W-Amplifier-rescue J2
 U 1 1 61C68424
 P 2200 4650
@@
 $EndComp
 $Comp
-L 70W-Amplifier-rescue:BNC-Xenir-70W-Amplifier-rescue-70W-Amplifier-rescue J1
+L 70W-Amplifier-rescue:BNC-Xenir-70W-Amplifier-rescue-70W-Amplifier-rescue-70W-Amplifier-rescue J1
 U 1 1 61C69914
 P 1800 4250
@@
 	5350 4350 5350 4450
 $Comp
-L 70W-Amplifier-rescue:Resistor-Xenir-70W-Amplifier-rescue-70W-Amplifier-rescue R3
+L 70W-Amplifier-rescue:Resistor-Xenir-70W-Amplifier-rescue-70W-Amplifier-rescue-70W-Amplifier-rescue R3
 U 1 1 61CCDCF5
 P 5700 4550
@@
 $EndComp
 $Comp
-L 70W-Amplifier-rescue:Capacitor-Xenir-70W-Amplifier-rescue-70W-Amplifier-rescue C3
+L 70W-Amplifier-rescue:Capacitor-Xenir-70W-Amplifier-rescue-70W-Amplifier-rescue-70W-Amplifier-rescue C3
 U 1 1 61CCE86F
 P 6050 4500
@@
 	5350 4950 6400 4950
 $Comp
-L 70W-Amplifier-rescue:Resistor-Xenir-70W-Amplifier-rescue-70W-Amplifier-rescue R4
+L 70W-Amplifier-rescue:Resistor-Xenir-70W-Amplifier-rescue-70W-Amplifier-rescue-70W-Amplifier-rescue R4
 U 1 1 61CDA054
 P 6750 3300
@@
 $EndComp
 $Comp
-L 70W-Amplifier-rescue:Capacitor-Xenir-70W-Amplifier-rescue-70W-Amplifier-rescue C4
+L 70W-Amplifier-rescue:Capacitor-Xenir-70W-Amplifier-rescue-70W-Amplifier-rescue-70W-Amplifier-rescue C4
 U 1 1 61CDADD3
 P 6400 3600
@@
 	6400 3950 6650 3950
 $Comp
-L 70W-Amplifier-rescue:Capacitor-Xenir-70W-Amplifier-rescue-70W-Amplifier-rescue C5
+L 70W-Amplifier-rescue:Capacitor-Xenir-70W-Amplifier-rescue-70W-Amplifier-rescue-70W-Amplifier-rescue C5
 U 1 1 61CDF56C
 P 6400 5350
@@
 $EndComp
 $Comp
-L 70W-Amplifier-rescue:Resistor-Xenir-70W-Amplifier-rescue-70W-Amplifier-rescue R5
+L 70W-Amplifier-rescue:Resistor-Xenir-70W-Amplifier-rescue-70W-Amplifier-rescue-70W-Amplifier-rescue R5
 U 1 1 61CDFD89
 P 6750 5700
@@
 	8200 4350 8200 4450
 $Comp
-L 70W-Amplifier-rescue:Capacitor-Xenir-70W-Amplifier-rescue-70W-Amplifier-rescue C1
+L 70W-Amplifier-rescue:Capacitor-Xenir-70W-Amplifier-rescue-70W-Amplifier-rescue-70W-Amplifier-rescue C1
 U 1 1 61CECBAC
 P 7850 4500
@@
 LPF
 $Comp
-L 70W-Amplifier-rescue:Inductor-Xenir-70W-Amplifier-rescue-70W-Amplifier-rescue L1
+L 70W-Amplifier-rescue:Inductor-Xenir-70W-Amplifier-rescue-70W-Amplifier-rescue-70W-Amplifier-rescue L1
 U 1 1 61D26F6D
 P 7850 4000
@@
 	6050 4350 6050 4250
 $Comp
-L 70W-Amplifier-rescue:Resistor-Xenir-70W-Amplifier-rescue-70W-Amplifier-rescue R6
+L 70W-Amplifier-rescue:Resistor-Xenir-70W-Amplifier-rescue-70W-Amplifier-rescue-70W-Amplifier-rescue R6
 U 1 1 61C90F87
 P 6400 4400
@@
 	6400 4950 6400 4600
 $Comp
-L 70W-Amplifier-rescue:Splitter_Center_Tap-Xenir-70W-Amplifier-rescue-70W-Amplifier-rescue T1
+L 70W-Amplifier-rescue:Splitter_Center_Tap-Xenir-70W-Amplifier-rescue-70W-Amplifier-rescue-70W-Amplifier-rescue T1
 U 1 1 61CE4121
 P 5000 3850
@@
 	5350 4850 5350 4950
 $Comp
-L 70W-Amplifier-rescue:2N3906-SMD-Xenir-70W-Amplifier-rescue-70W-Amplifier-rescue Q1
+L 70W-Amplifier-rescue:2N3906-SMD-Xenir-70W-Amplifier-rescue-70W-Amplifier-rescue-70W-Amplifier-rescue Q1
 U 1 1 61CF1527
 P 5300 1800
@@
 $EndComp
 $Comp
-L 70W-Amplifier-rescue:PCB_SMA_EDGE-Xenir-70W-Amplifier-rescue-70W-Amplifier-rescue J3
+L 70W-Amplifier-rescue:PCB_SMA_EDGE-Xenir-70W-Amplifier-rescue-70W-Amplifier-rescue-70W-Amplifier-rescue J3
 U 1 1 61CF5952
 P 9650 4350
@@
 $EndComp
 $Comp
-L 70W-Amplifier-rescue:PCB_SMA_EDGE-Xenir-70W-Amplifier-rescue-70W-Amplifier-rescue J4
+L 70W-Amplifier-rescue:PCB_SMA_EDGE-Xenir-70W-Amplifier-rescue-70W-Amplifier-rescue-70W-Amplifier-rescue J4
 U 1 1 61CF9C6B
 P 10500 4350
@@
 $EndComp
 $Comp
-L 70W-Amplifier-rescue:Splitter_Center_Tap-Xenir-70W-Amplifier-rescue-70W-Amplifier-rescue T2
+L 70W-Amplifier-rescue:Splitter_Center_Tap-Xenir-70W-Amplifier-rescue-70W-Amplifier-rescue-70W-Amplifier-rescue T2
 U 1 1 61CFF29A
 P 8550 5050
@@
 Q3Drain
 $Comp
-L 70W-Amplifier-rescue:Resistor-Xenir-70W-Amplifier-rescue-70W-Amplifier-rescue R8
+L 70W-Amplifier-rescue:Resistor-Xenir-70W-Amplifier-rescue-70W-Amplifier-rescue-70W-Amplifier-rescue R8
 U 1 1 61E660AB
 P 7150 4150
@@
 $EndComp
 $Comp
-L 70W-Amplifier-rescue:Resistor-Xenir-70W-Amplifier-rescue-70W-Amplifier-rescue R9
+L 70W-Amplifier-rescue:Resistor-Xenir-70W-Amplifier-rescue-70W-Amplifier-rescue-70W-Amplifier-rescue R9
 U 1 1 61E6F0FA
 P 7150 4750
@@
 $EndComp
 $Comp
-L 70W-Amplifier-rescue:Capacitor-Xenir-70W-Amplifier-rescue-70W-Amplifier-rescue C6
+L 70W-Amplifier-rescue:Capacitor-Xenir-70W-Amplifier-rescue-70W-Amplifier-rescue-70W-Amplifier-rescue C6
 U 1 1 61E6FCAB
 P 7100 4325
@@
 $EndComp
 $Comp
-L 70W-Amplifier-rescue:Capacitor-Xenir-70W-Amplifier-rescue-70W-Amplifier-rescue C7
+L 70W-Amplifier-rescue:Capacitor-Xenir-70W-Amplifier-rescue-70W-Amplifier-rescue-70W-Amplifier-rescue C7
 U 1 1 61E706E7
 P 7100 4550
@@
 	7350 4550 7350 4450
 $Comp
-L 70W-Amplifier-rescue:Capacitor-Xenir-70W-Amplifier-rescue-70W-Amplifier-rescue C8
+L 70W-Amplifier-rescue:Capacitor-Xenir-70W-Amplifier-rescue-70W-Amplifier-rescue-70W-Amplifier-rescue C8
 U 1 1 61E9AE04
 P 9050 4750
