File: 70W-Amplifier.kicad_pcb (KiCad board)
At the start: 2 copper layers, 31 parts, among them J1 RF_OUT, J2 RF_IN, J3 LPF_IN, J4 LPF_OUT, J5 13.8V Input, J6 PTT, K1 G5V-2, Q1 2N3906, Q2 IRF530, Q3 IRF530, T1 BN43-202 2T:1T, T2 FERRITE TUBE 1T:3T, U1 L7805

Commit message: Update 70W-Amplifier.kicad_pcb
Other:
- board outline added: 103.3 x 60.5 mm

Commit message: still going
Parts:
- J1, J2: footprint Connector_Coaxial:SMA_Amphenol_132289_EdgeMount -> Xenir:BNC
- U1: footprint Package_TO_SOT_SMD:SOT-223-3_TabPin2 -> Package_TO_SOT_SMD:TO-252-3_TabPin2
- moved J1 49.2 mm to (121.9, 63.9)
- moved J2 35.5 mm to (142.4, 63.9)
- moved U1 35.5 mm to (186.3, 81.0)
Connections:
- K1 pad 9: Net-(K1-Pad9) -> (no net)

Commit message: added splitter
Parts:
- J3, J4: footprint Connector_Coaxial:SMA_Amphenol_132289_EdgeMount -> Xenir:PCB-SMA-EDGE
- Q1: value 2N3906 -> 2N3906-SMD; footprint Package_TO_SOT_THT:TO-92_Inline -> Package_TO_SOT_SMD:SOT-23
- T1: value BN43-202 2T:1T -> BN-43-202 1T:2T; footprint Xenir:BN-43-202-Vertical -> Xenir:BN-43-202-Splitter-SMD
- T2: value FERRITE TUBE 1T:3T -> Ferrite 1T:3T; footprint Xenir:BN-43-202-Vertical -> Xenir:Ferrite-Tube-Splitter-SMD
- moved T2 75.1 mm to (202.1, 141.2)
- moved Q1 48.5 mm to (187.8, 128.4)
- moved T1 31.4 mm to (139.6, 134.5)
- moved J4 19.0 mm to (136.2, 85.8)
- moved J3 7.05 mm to (128.8, 85.8)
Connections:
- K1 pad 9: (no net) -> Net-(K1-Pad9)
- Q1 pad 1: +12V -> Net-(Q1-Pad1)
- Q1 pad 2: Net-(Q1-Pad2) -> TRANSMIT_ON
- Q1 pad 3: TRANSMIT_ON -> +12V
- R1 pad 1: Net-(Q1-Pad2) -> Net-(Q1-Pad1)
- R2 pad 2: Net-(Q1-Pad2) -> Net-(Q1-Pad1)
- T1 pad 1: (no net) -> GND
- T1 pad 2: (no net) -> Net-(K1-Pad9)
- T2 pad 1: (no net) -> GND
- T2 pad 2: (no net) -> Net-(J3-Pad1)

Commit message: pcb work
Parts:
- J5: footprint Xenir:Power Connector -> Connector_BarrelJack:BarrelJack_Horizontal
- moved U1 124.3 mm to (81.0, 147.1), turned to 90 degrees
- moved Q1 122.0 mm to (67.3, 147.6), turned to 270 degrees
- moved R2 108.3 mm to (71.9, 140.0)
- moved R1 100.8 mm to (75.3, 147.3), turned to 270 degrees
- moved J1 100.7 mm to (48.3, 132.6), turned to 90 degrees
- moved J2 98.2 mm to (48.5, 92.7), turned to 90 degrees
- moved EC1 94.9 mm to (68.6, 158.0), turned to 90 degrees
- moved J3 87.3 mm to (149.4, 170.7), turned to 270 degrees
- moved J4 85.3 mm to (125.4, 170.5), turned to 270 degrees
- moved J5 70.5 mm to (55.6, 157.5)
- moved T1 57.4 mm to (97.6, 95.3)
- moved JP1 49.2 mm to (132.1, 161.0), turned to 180 degrees
- moved K1 39.3 mm to (68.8, 104.4)
- moved D1 31.2 mm to (76.5, 99.6), turned to 180 degrees
Other:
- board outline removed

Commit message: added resistors
Parts:
- R4, R5, R6: footprint Xenir:Resistor 1206 -> Resistor_THT:R_Axial_DIN0414_L11.9mm_D4.5mm_P20.32mm_Horizontal
- moved C1 78.2 mm to (239.0, 79.5)
- moved L1 71.1 mm to (205.2, 60.5), turned to 90 degrees
- moved J4 60.9 mm to (137.6, 110.8)
- moved J3 60.9 mm to (161.5, 111.0)
- moved JP1 60.9 mm to (144.3, 101.3)
- moved C2 59.0 mm to (140.6, 60.0)
- moved Q1 56.3 mm to (104.9, 105.7)
- moved R1 56.3 mm to (112.9, 105.4)
- moved R2 56.3 mm to (109.5, 98.0)
- moved EC1 56.3 mm to (106.2, 116.1)
- moved U1 56.3 mm to (118.6, 105.2)
- moved R7 52.5 mm to (129.5, 67.8), turned to 90 degrees
- moved J1 51.4 mm to (85.3, 96.9)
- moved EC2 50.3 mm to (123.2, 67.8), turned to 270 degrees
- moved T1 49.3 mm to (140.5, 70.9)
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Connections:
- net Net-(Q2-Pad2) renamed /Q2Drain
- net Net-(Q3-Pad2) renamed /Q3Drain
- T1 pad 1: GND -> Net-(K1-Pad9)
- T1 pad 2: Net-(K1-Pad9) -> GND
Routing:
- net GND: track 20.7 -> 0.00 mm
Other:
- board outline added: 168.1 x 104.6 mm

Commit message: Update 70W-Amplifier.kicad_pcb
Parts:
- moved J5 16.0 mm to (91.9, 116.6)
- moved R4 13.7 mm to (185.2, 53.3)
- moved R5 13.7 mm to (185.7, 111.3)
- moved C5 6.64 mm to (158.6, 101.9)
- moved Q2 0.40 mm to (175.0, 66.2)
- moved Q3 0.33 mm to (175.5, 98.4)
Other:
- outline, holes or cut-outs redrawn

Commit message: added source resistor/cap
Parts:
- added C6: .2uF, Xenir:Capacitor 1206, F.Cu at (157.9, 52.9)
- added C7: .2uF, Xenir:Capacitor 1206, F.Cu at (195.2, 111.7)
- added R8: .17, Resistor_SMD:R_2512_6332Metric, F.Cu at (157.6, 59.7)
- added R9: .17, Resistor_SMD:R_2512_6332Metric, F.Cu at (195.1, 104.6)
Connections:
- Q2 pad 3: GND -> Net-(C6-Pad2)
- Q3 pad 3: GND -> Net-(C7-Pad2)

Commit message: gg
Parts:
- moved J5 132.6 mm to (223.9, 103.7), turned to 90 degrees
- moved L1 57.1 mm to (209.3, 117.4), turned to 180 degrees
- moved C7 2.41 mm to (197.5, 112.5)
- moved R9 2.41 mm to (197.4, 105.4)
- moved R5 2.05 mm to (185.9, 113.3)
- moved R4 1.78 mm to (185.2, 51.6)
Routing:
- net Net-(C1-Pad1): track 0.00 -> 34.0 mm
- net /Q2Drain: track 0.00 -> 30.3 mm
- net /Q3Drain: track 0.00 -> 29.5 mm
- net +12V: track 0.00 -> 15.7 mm
Other:
- board outline removed
