File: 70W-Amplifier.kicad_pcb (KiCad board)
At the start: 2 copper layers, 35 parts, among them J1 RF_OUT, J2 RF_IN, J3 LPF_IN, J4 LPF_OUT, J5 13.8V Input, J6 PTT, K1 G5V-2, Q1 2N3906-SMD, Q2 IRF530, Q3 IRF530, T1 BN-43-202 1T:2T, T2 Ferrite 1T:3T, U1 L7805

Commit message: Update 70W-Amplifier.kicad_pcb
Parts:
- moved R9 23.0 mm to (175.8, 113.3), turned to 180 degrees
- moved C7 21.9 mm to (175.8, 115.6), turned to 0 degrees
- moved R8 18.6 mm to (175.2, 53.6), turned to 0 degrees
- moved C6 17.7 mm to (175.5, 52.1), turned to 180 degrees
- moved R5 16.3 mm to (185.4, 97.0)
- moved R4 16.3 mm to (185.4, 67.8)
- moved J1 1.85 mm to (83.5, 97.4)
- moved J2 1.85 mm to (83.6, 68.3)
Connections:
- T2 pad 1: GND -> Net-(J3-Pad1)
- T2 pad 2: Net-(J3-Pad1) -> GND
Routing:
- net Net-(C7-Pad2): track 0.00 -> 14.5 mm
- net Net-(C6-Pad2): track 0.00 -> 11.4 mm
Other:
- board outline added: 169.7 x 77.7 mm
Changed lines of the file:
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@@
   (general
     (thickness 1.6)
-    (drawings 0)
-    (tracks 15)
+    (drawings 8)
+    (tracks 26)
     (zones 0)
     (modules 35)
@@
   )
   (module Resistor_SMD:R_2512_6332Metric (layer F.Cu)
-    (at 197.358 105.41)
+    (at 175.768 113.284 180)
     (descr "Resistor SMD 2512 (6332 Metric), square (rectangular) end terminal, IPC_7351 nominal, (Body size source: IPC-SM-782 page 72, https://www.pcb-3d.com/wordpress/wp-content/uploads/ipc-sm-782a_amendment_1_and_2.pdf), generated with kicad-footprint-generator")
     (tags resistor)
@@
       (effects (font (size 1 1) (thickness 0.15)))
     )
-    (pad 2 smd roundrect (at 2.9625 0) (size 1.225 3.35) (layers F.Cu F.Paste F.Mask) (roundrect_rratio 0.204082)
-      (net 1 GND))
-    (pad 1 smd roundrect (at -2.9625 0) (size 1.225 3.35) (layers F.Cu F.Paste F.Mask) (roundrect_rratio 0.204082)
+    (pad 2 smd roundrect (at 2.9625 0 180) (size 1.225 3.35) (layers F.Cu F.Paste F.Mask) (roundrect_rratio 0.204082)
+      (net 1 GND))
+    (pad 1 smd roundrect (at -2.9625 0 180) (size 1.225 3.35) (layers F.Cu F.Paste F.Mask) (roundrect_rratio 0.204082)
       (net 23 "Net-(C7-Pad2)"))
     (model ${KISYS3DMOD}/Resistor_SMD.3dshapes/R_2512_6332Metric.wrl
@@
   )
   (module Resistor_SMD:R_2512_6332Metric (layer F.Cu)
-    (at 157.6485 59.69 180)
+    (at 175.1745 53.594)
     (descr "Resistor SMD 2512 (6332 Metric), square (rectangular) end terminal, IPC_7351 nominal, (Body size source: IPC-SM-782 page 72, https://www.pcb-3d.com/wordpress/wp-content/uploads/ipc-sm-782a_amendment_1_and_2.pdf), generated with kicad-footprint-generator")
     (tags resistor)
@@
       (effects (font (size 1 1) (thickness 0.15)))
     )
-    (pad 2 smd roundrect (at 2.9625 0 180) (size 1.225 3.35) (layers F.Cu F.Paste F.Mask) (roundrect_rratio 0.204082)
-      (net 1 GND))
-    (pad 1 smd roundrect (at -2.9625 0 180) (size 1.225 3.35) (layers F.Cu F.Paste F.Mask) (roundrect_rratio 0.204082)
+    (pad 2 smd roundrect (at 2.9625 0) (size 1.225 3.35) (layers F.Cu F.Paste F.Mask) (roundrect_rratio 0.204082)
+      (net 1 GND))
+    (pad 1 smd roundrect (at -2.9625 0) (size 1.225 3.35) (layers F.Cu F.Paste F.Mask) (roundrect_rratio 0.204082)
       (net 22 "Net-(C6-Pad2)"))
     (model ${KISYS3DMOD}/Resistor_SMD.3dshapes/R_2512_6332Metric.wrl
@@
   )
   (module "Xenir:Capacitor 1206" (layer F.Cu)
-    (at 197.482 112.486 180)
+    (at 175.768 115.57)
     (fp_text reference C7 (at 0 0.5) (layer F.SilkS)
       (effects (font (size 0.5 0.5) (thickness 0.125)))
@@
       (effects (font (size 0.8 0.8) (thickness 0.12)))
     )
-    (pad 2 smd roundrect (at 1.4 2.25 180) (size 1.25 1.75) (layers F.Cu F.Paste F.Mask) (roundrect_rratio 0.2)
+    (pad 2 smd roundrect (at 1.4 2.25) (size 1.25 1.75) (layers F.Cu F.Paste F.Mask) (roundrect_rratio 0.2)
       (net 23 "Net-(C7-Pad2)"))
-    (pad 1 smd roundrect (at -1.4 2.25 180) (size 1.25 1.75) (layers F.Cu F.Paste F.Mask) (roundrect_rratio 0.2)
+    (pad 1 smd roundrect (at -1.4 2.25) (size 1.25 1.75) (layers F.Cu F.Paste F.Mask) (roundrect_rratio 0.2)
       (net 1 GND))
   )
   (module "Xenir:Capacitor 1206" (layer F.Cu)
-    (at 157.858 52.868)
+    (at 175.514 52.07 180)
     (fp_text reference C6 (at 0 0.5) (layer F.SilkS)
       (effects (font (size 0.5 0.5) (thickness 0.125)))
@@
       (effects (font (size 0.8 0.8) (thickness 0.12)))
     )
-    (pad 2 smd roundrect (at 1.4 2.25) (size 1.25 1.75) (layers F.Cu F.Paste F.Mask) (roundrect_rratio 0.2)
+    (pad 2 smd roundrect (at 1.4 2.25 180) (size 1.25 1.75) (layers F.Cu F.Paste F.Mask) (roundrect_rratio 0.2)
       (net 22 "Net-(C6-Pad2)"))
-    (pad 1 smd roundrect (at -1.4 2.25) (size 1.25 1.75) (layers F.Cu F.Paste F.Mask) (roundrect_rratio 0.2)
+    (pad 1 smd roundrect (at -1.4 2.25 180) (size 1.25 1.75) (layers F.Cu F.Paste F.Mask) (roundrect_rratio 0.2)
       (net 1 GND))
   )
@@
   )
   (module Resistor_THT:R_Axial_DIN0414_L11.9mm_D4.5mm_P20.32mm_Horizontal (layer F.Cu)
-    (at 185.928 113.284 180)
+    (at 185.42 97.028 180)
     (descr "Resistor, Axial_DIN0414 series, Axial, Horizontal, pin pitch=20.32mm, 2W, length*diameter=11.9*4.5mm^2, http://www.vishay.com/docs/20128/wkxwrx.pdf")
     (tags "Resistor Axial_DIN0414 series Axial Horizontal pin pitch 20.32mm 2W length 11.9mm diameter 4.5mm")
@@
   )
   (module Resistor_THT:R_Axial_DIN0414_L11.9mm_D4.5mm_P20.32mm_Horizontal (layer F.Cu)
-    (at 185.166 51.562 180)
+    (at 185.42 67.818 180)
     (descr "Resistor, Axial_DIN0414 series, Axial, Horizontal, pin pitch=20.32mm, 2W, length*diameter=11.9*4.5mm^2, http://www.vishay.com/docs/20128/wkxwrx.pdf")
     (tags "Resistor Axial_DIN0414 series Axial Horizontal pin pitch 20.32mm 2W length 11.9mm diameter 4.5mm")
@@
       (net 21 /Q3Drain))
     (pad 2 smd rect (at -18.1 28.6 180) (size 4 4) (layers F.Cu F.Paste F.Mask)
-      (net 12 "Net-(J3-Pad1)"))
+      (net 1 GND))
     (pad 4 smd rect (at -18.2 17.3 180) (size 4 4) (layers F.Cu F.Paste F.Mask)
       (net 2 "Net-(C1-Pad1)"))
     (pad 1 smd rect (at -18.2 6.7 180) (size 4 4) (layers F.Cu F.Paste F.Mask)
-      (net 1 GND))
+      (net 12 "Net-(J3-Pad1)"))
   )
   (module Xenir:PCB-SMA-EDGE (layer F.Cu)
@@
   )
   (module Xenir:BNC (layer F.Cu)
-    (at 85.344 67.818 90)
+    (at 83.566 68.326 90)
     (fp_text reference J2 (at 0.7 -3 90) (layer F.SilkS)
       (effects (font (size 1 1) (thickness 0.15)))
@@
   )
   (module Xenir:BNC (layer F.Cu)
-    (at 85.254 96.928 90)
+    (at 83.476 97.436 90)
     (fp_text reference J1 (at 0.7 -3 90) (layer F.SilkS)
       (effects (font (size 1 1) (thickness 0.15)))
@@
       (net 2 "Net-(C1-Pad1)"))
   )
+  (gr_line (start 184.404 73.914) (end 184.404 91.44) (layer Edge.Cuts) (width 0.1))
+  (gr_line (start 167.386 73.914) (end 184.404 73.914) (layer Edge.Cuts) (width 0.1))
+  (gr_line (start 167.386 91.44) (end 167.386 73.914) (layer Edge.Cuts) (width 0.1))
+  (gr_line (start 184.404 91.44) (end 167.386 91.44) (layer Edge.Cuts) (width 0.1))
+  (gr_line (start 246.38 45.974) (end 246.38 123.698) (layer Edge.Cuts) (width 0.1))
+  (gr_line (start 76.708 45.974) (end 246.38 45.974) (layer Edge.Cuts) (width 0.1))
+  (gr_line (start 76.708 123.698) (end 76.708 45.974) (layer Edge.Cuts) (width 0.1))
+  (gr_line (start 246.38 123.698) (end 76.708 123.698) (layer Edge.Cuts) (width 0.1))
   (segment (start 233.084 82.892) (end 209.296 106.68) (width 3) (layer F.Cu) (net 2))
   (segment (start 233.084 82.522) (end 233.084 82.892) (width 3) (layer F.Cu) (net 2))
@@
   (segment (start 175.19904 60.198) (end 175.19904 62.67704) (width 2) (layer F.Cu) (net 20))
   (segment (start 175.19904 62.67704) (end 176.53 64.008) (width 2) (layer F.Cu) (net 20))
-  (segment (start 176.53 64.008) (end 189.484 64.008) (width 2) (layer F.Cu) (net 20))
   (segment (start 193.384 67.908) (end 193.384 75.422) (width 2) (layer F.Cu) (net 20))
   (segment (start 189.484 64.008) (end 193.384 67.908) (width 2) (layer F.Cu) (net 20))
+  (segment (start 185.42 64.008) (end 189.484 64.008) (width 2) (layer F.Cu) (net 20))
+  (segment (start 176.53 64.008) (end 185.42 64.008) (width 2) (layer F.Cu) (net 20))
   (segment (start 193.384 89.222) (end 193.384 95.922) (width 2) (layer F.Cu) (net 21))
   (segment (start 193.384 95.922) (end 189.738 99.568) (width 2) (layer F.Cu) (net 21))
   (segment (start 175.26 102.388838) (end 175.26 104.394) (width 2) (layer F.Cu) (net 21))
   (segment (start 178.080838 99.568) (end 175.26 102.388838) (width 2) (layer F.Cu) (net 21))
-  (segment (start 189.738 99.568) (end 178.080838 99.568) (width 2) (layer F.Cu) (net 21))
+  (segment (start 185.928 99.822) (end 185.674 99.568) (width 2) (layer F.Cu) (net 21))
+  (segment (start 185.674 99.568) (end 178.080838 99.568) (width 2) (layer F.Cu) (net 21))
+  (segment (start 189.738 99.568) (end 185.674 99.568) (width 2) (layer F.Cu) (net 21))
+  (segment (start 172.6692 54.0512) (end 172.212 53.594) (width 2) (layer F.Cu) (net 22))
+  (segment (start 172.6692 60.198) (end 172.6692 54.0512) (width 2) (layer F.Cu) (net 22))
+  (segment (start 174.114 51.692) (end 172.212 53.594) (width 2) (layer F.Cu) (net 22))
+  (segment (start 174.114 49.82) (end 174.114 51.692) (width 2) (layer F.Cu) (net 22))
+  (segment (start 177.78984 112.34334) (end 178.7305 113.284) (width 2) (layer F.Cu) (net 23))
+  (segment (start 177.78984 104.394) (end 177.78984 112.34334) (width 2) (layer F.Cu) (net 23))
+  (segment (start 178.7305 116.2575) (end 177.168 117.82) (width 2) (layer F.Cu) (net 23))
+  (segment (start 178.7305 113.284) (end 178.7305 116.2575) (width 2) (layer F.Cu) (net 23))
 )

Commit message: finished pcb
Parts:
- moved EC1 94.5 mm to (200.7, 113.0)
- moved C5 6.39 mm to (158.8, 95.5)
- moved R4 6.36 mm to (185.2, 61.5)
- moved R5 5.84 mm to (185.4, 102.9)
Routing:
- net +12V: track 15.7 -> 131.6 mm
- net Net-(J3-Pad1): track 0.00 -> 104.9 mm, vias 0 -> 2
- net LPF: track 0.00 -> 73.0 mm, vias 0 -> 2
- net Net-(EC2-Pad1): track 0.00 -> 57.7 mm
- net TRANSMIT_ON: track 0.00 -> 55.0 mm
- net Net-(C4-Pad2): track 0.00 -> 47.4 mm, vias 0 -> 2
- net Net-(J1-PadS): track 0.00 -> 40.0 mm
- net Net-(K1-Pad9): track 0.00 -> 39.5 mm, vias 0 -> 2
- net BIAS: track 0.00 -> 38.1 mm
- net Net-(C5-Pad1): track 0.00 -> 36.1 mm
- net Net-(J2-PadS): track 0.00 -> 16.4 mm
- net Net-(C2-Pad1): track 0.00 -> 14.2 mm
- net Net-(C4-Pad1): track 0.00 -> 8.86 mm
- net Net-(Q1-Pad1): track 0.00 -> 8.53 mm
- net Net-(C5-Pad2): track 0.00 -> 8.21 mm
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- added copper zone on B.Cu, net GND
- added copper zone on F.Cu, net GND
Other:
- board size 169.7 x 77.7 mm -> 170.9 x 81 mm

Commit message: gg
Parts:
- VR1: footprint Xenir:Trimpot Vertical -> Xenir:Trimpot_Horizontal_SMD
- moved VR1 2.20 mm to (135.6, 70.4)
- moved C2 0.51 mm to (140.6, 60.5)
Routing:
- net Net-(C2-Pad1): track 14.2 -> 18.5 mm
- removed copper zone on B.Cu, net GND
- removed copper zone on F.Cu, net GND

Commit message: changed to surface mount
Parts:
- K1: footprint Relay_THT:Relay_DPDT_Omron_G5V-2 -> Xenir:Relay_DPDT_Omron_G5V-2-SMD
- moved K1 2.54 mm to (107.4, 79.8)
Routing:
- net Net-(J2-PadS): track 16.4 -> 11.6 mm
- net Net-(K1-Pad9): track 39.5 -> 44.3 mm
- net GND: track 4.83 -> 0.00 mm
- net Net-(K1-Pad11): track 7.62 -> 12.2 mm
- net TRANSMIT_ON: track 55.0 -> 57.0 mm
- net Net-(J1-PadS): track 40.0 -> 41.7 mm

Commit message: finished
Parts:
- L1: footprint Xenir:BN-43-202-Vertical -> Xenir:BN-43-202-Vertical-SMD
- R4, R5, R6: footprint Resistor_THT:R_Axial_DIN0414_L11.9mm_D4.5mm_P20.32mm_Horizontal -> Xenir:LargeResistorSurfaceMount
- moved C6 14.6 mm to (161.7, 47.5), turned to 0 degrees
- moved R8 7.06 mm to (169.1, 50.0)
- moved C7 5.46 mm to (181.2, 115.5), turned to 180 degrees
- moved Q2 3.84 mm to (174.5, 62.3)
- moved R4 3.82 mm to (184.9, 57.7)
- moved L1 3.58 mm to (212.9, 117.9)
- moved R5 3.31 mm to (185.7, 106.2)
- moved Q3 2.60 mm to (174.9, 101.0)
- moved R9 1.78 mm to (174.0, 113.3)
Routing:
- net Net-(C6-Pad2): track 11.4 -> 6.15 mm
- net /Q2Drain: track 33.0 -> 37.4 mm
- net /Q3Drain: track 32.9 -> 37.1 mm
- net Net-(C7-Pad2): track 14.5 -> 10.5 mm
- net Net-(C5-Pad1): track 36.1 -> 39.1 mm
- net Net-(C4-Pad2): track 47.4 -> 50.4 mm
- net Net-(C5-Pad2): track 8.21 -> 10.6 mm
- net Net-(C4-Pad1): track 8.86 -> 11.1 mm
- net +12V: track 131.6 -> 129.5 mm
- net Net-(C1-Pad1): track 38.9 -> 38.3 mm
- added copper zone on B.Cu, net GND
- added copper zone on F.Cu, net GND
Other:
- outline, holes or cut-outs redrawn

Commit message: Update 70W-Amplifier.kicad_pcb
Parts:
- moved C6 6.00 mm to (167.7, 47.5)
- moved R8 6.00 mm to (175.1, 50.0)
Routing:
- net Net-(C6-Pad2): track 6.15 -> 15.7 mm
- net +12V: track 129.5 -> 133.3 mm

Commit message: added gerber
Parts:
- J5: footprint Connector_BarrelJack:BarrelJack_Horizontal -> Xenir:PowerConnectorPads
- J6: footprint Xenir:Power Connector -> Xenir:TwoPads
- moved J5 12.9 mm to (227.5, 116.1), turned to 180 degrees
- moved J6 1.54 mm to (112.3, 95.4)
Changed lines of the file:
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@@
-(kicad_pcb (version 20171130) (host pcbnew 5.1.12-unknown-nightly-202112011503)
+(kicad_pcb (version 20171130) (host pcbnew "(5.1.5)-3")
   (general
     (thickness 1.6)
@@
   )
   (setup
-    (last_trace_width 1)
+    (last_trace_width 0.25)
     (user_trace_width 1)
     (user_trace_width 2)
@@
     (pcbplotparams
       (layerselection 0x010fc_ffffffff)
-      (usegerberextensions false)
-      (usegerberattributes true)
-      (usegerberadvancedattributes true)
-      (creategerberjobfile true)
+      (usegerberextensions true)
+      (usegerberattributes false)
+      (usegerberadvancedattributes false)
+      (creategerberjobfile false)
       (excludeedgelayer true)
       (linewidth 0.100000)
@@
       (psa4output false)
       (plotreference true)
-      (plotvalue true)
+      (plotvalue false)
       (plotinvisibletext false)
       (padsonsilk false)
-      (subtractmaskfromsilk false)
-      (outputformat 4)
+      (subtractmaskfromsilk true)
+      (outputformat 1)
       (mirror false)
       (drillshape 0)
       (scaleselection 1)
-      (outputdirectory "/home/xenir/kicad/70W-Amplifier/"))
+      (outputdirectory "C:/Users/Caliphax/Documents/70W-Amplifier/gerber/"))
   )
   (net 0 "")
@@
     (add_net TRANSMIT_ON)
   )
+  (module Xenir:TwoPads (layer F.Cu)
+    (at 112.3 95.4 270)
+    (fp_text reference J6 (at 0.5588 1.15316 90) (layer F.SilkS)
+      (effects (font (size 1 1) (thickness 0.15)))
+    )
+    (fp_text value PTT (at -4.65836 5.10032) (layer F.Fab)
+      (effects (font (size 1 1) (thickness 0.15)))
+    )
+    (fp_text user %R (at 0.67564 9.13638 90) (layer F.Fab)
+      (effects (font (size 0.98 0.98) (thickness 0.15)))
+    )
+    (fp_line (start -3.5687 2.2225) (end -3.5687 8.1025) (layer F.CrtYd) (width 0.05))
+    (fp_line (start 2.77114 8.11022) (end -3.57886 8.11022) (layer F.CrtYd) (width 0.05))
+    (fp_line (start 2.7686 2.22758) (end -3.5814 2.22758) (layer F.CrtYd) (width 0.05))
+    (fp_line (start 2.7686 2.22758) (end 2.7686 8.10758) (layer F.CrtYd) (width 0.05))
+    (pad 2 smd roundrect (at -0.3 4 270) (size 5 1.4) (layers F.Cu F.Paste F.Mask) (roundrect_rratio 0.25)
+      (net 14 "Net-(J6-Pad2)"))
+    (pad 1 smd roundrect (at -0.3 6.4 270) (size 5 1.4) (layers F.Cu F.Paste F.Mask) (roundrect_rratio 0.25)
+      (net 1 GND))
+  )
+  (module Xenir:PowerConnectorPads (layer F.Cu)
+    (at 227.5 116.1 180)
+    (fp_text reference J5 (at 0.4 2.2) (layer F.SilkS)
+      (effects (font (size 1 1) (thickness 0.15)))
+    )
+    (fp_text value "13.8V Input" (at 0.3 0.5) (layer F.Fab)
+      (effects (font (size 1 1) (thickness 0.15)))
+    )
+    (fp_text user VCC (at 3.5 4.1) (layer F.SilkS)
+      (effects (font (size 1 1) (thickness 0.15)))
+    )
+    (fp_text user GND (at -3.6 4.2) (layer F.SilkS)
+      (effects (font (size 1 1) (thickness 0.15)))
+    )
+    (pad 2 smd circle (at 3.6 6.5 180) (size 3 3) (layers F.Cu F.Paste F.Mask)
+      (net 10 +12V))
+    (pad 1 smd circle (at -3.5 6.6 180) (size 3 3) (layers F.Cu F.Paste F.Mask)
+      (net 1 GND))
+  )
   (module Xenir:BN-43-202-Vertical-SMD (layer F.Cu)
     (at 212.852 117.856 180)
@@
     (model ${KISYS3DMOD}/Package_TO_SOT_THT.3dshapes/TO-220-3_Horizontal_TabDown.wrl
       (offset (xyz -2.575 -6 0))
-      (scale (xyz 1 1 1))
-      (rotate (xyz 0 0 0))
-    )
-  )
-  (module Connector_BarrelJack:BarrelJack_Horizontal (layer F.Cu)
-    (at 223.9 103.68 90)
-    (descr "DC Barrel Jack")
-    (tags "Power Jack")
-    (fp_text reference J5 (at -8.45 5.75 90) (layer F.SilkS)
-      (effects (font (size 1 1) (thickness 0.15)))
-    )
-    (fp_text value "13.8V Input" (at -6.2 -5.5 90) (layer F.Fab)
-      (effects (font (size 1 1) (thickness 0.15)))
-    )
-    (fp_line (start 0 -4.5) (end -13.7 -4.5) (layer F.Fab) (width 0.1))
-    (fp_line (start 0.8 4.5) (end 0.8 -3.75) (layer F.Fab) (width 0.1))
-    (fp_line (start -13.7 4.5) (end 0.8 4.5) (layer F.Fab) (width 0.1))
-    (fp_line (start -13.7 -4.5) (end -13.7 4.5) (layer F.Fab) (width 0.1))
-    (fp_line (start -10.2 -4.5) (end -10.2 4.5) (layer F.Fab) (width 0.1))
-    (fp_line (start 0.9 -4.6) (end 0.9 -2) (layer F.SilkS) (width 0.12))
-    (fp_line (start -13.8 -4.6) (end 0.9 -4.6) (layer F.SilkS) (width 0.12))
-    (fp_line (start 0.9 4.6) (end -1 4.6) (layer F.SilkS) (width 0.12))
-    (fp_line (start 0.9 1.9) (end 0.9 4.6) (layer F.SilkS) (width 0.12))
-    (fp_line (start -13.8 4.6) (end -13.8 -4.6) (layer F.SilkS) (width 0.12))
-    (fp_line (start -5 4.6) (end -13.8 4.6) (layer F.SilkS) (width 0.12))
-    (fp_line (start -14 4.75) (end -14 -4.75) (layer F.CrtYd) (width 0.05))
-    (fp_line (start -5 4.75) (end -14 4.75) (layer F.CrtYd) (width 0.05))
-    (fp_line (start -5 6.75) (end -5 4.75) (layer F.CrtYd) (width 0.05))
-    (fp_line (start -1 6.75) (end -5 6.75) (layer F.CrtYd) (width 0.05))
-    (fp_line (start -1 4.75) (end -1 6.75) (layer F.CrtYd) (width 0.05))
-    (fp_line (start 1 4.75) (end -1 4.75) (layer F.CrtYd) (width 0.05))
-    (fp_line (start 1 2) (end 1 4.75) (layer F.CrtYd) (width 0.05))
-    (fp_line (start 2 2) (end 1 2) (layer F.CrtYd) (width 0.05))
-    (fp_line (start 2 -2) (end 2 2) (layer F.CrtYd) (width 0.05))
-    (fp_line (start 1 -2) (end 2 -2) (layer F.CrtYd) (width 0.05))
-    (fp_line (start 1 -4.5) (end 1 -2) (layer F.CrtYd) (width 0.05))
-    (fp_line (start 1 -4.75) (end -14 -4.75) (layer F.CrtYd) (width 0.05))
-    (fp_line (start 1 -4.5) (end 1 -4.75) (layer F.CrtYd) (width 0.05))
-    (fp_line (start 0.05 -4.8) (end 1.1 -4.8) (layer F.SilkS) (width 0.12))
-    (fp_line (start 1.1 -3.75) (end 1.1 -4.8) (layer F.SilkS) (width 0.12))
-    (fp_line (start -0.003213 -4.505425) (end 0.8 -3.75) (layer F.Fab) (width 0.1))
-    (fp_text user %R (at -3 -2.95 90) (layer F.Fab)
-      (effects (font (size 1 1) (thickness 0.15)))
-    )
-    (pad 3 thru_hole roundrect (at -3 4.7 90) (size 3.5 3.5) (drill oval 3 1) (layers *.Cu *.Mask) (roundrect_rratio 0.25))
-    (pad 2 thru_hole roundrect (at -6 0 90) (size 3 3.5) (drill oval 1 3) (layers *.Cu *.Mask) (roundrect_rratio 0.25)
-      (net 10 +12V))
-    (pad 1 thru_hole rect (at 0 0 90) (size 3.5 3.5) (drill oval 1 3) (layers *.Cu *.Mask)
-      (net 1 GND))
-    (model ${KISYS3DMOD}/Connector_BarrelJack.3dshapes/BarrelJack_Horizontal.wrl
-      (at (xyz 0 0 0))
       (scale (xyz 1 1 1))
       (rotate (xyz 0 0 0))
@@
     (pad 1 smd rect (at -1.75 1.25 180) (size 3.25 1.5) (layers F.Cu F.Mask)
       (net 12 "Net-(J3-Pad1)"))
-  )
-  (module "Xenir:Power Connector" (layer F.Cu)
-    (at 113.538 94.488 270)
-    (fp_text reference J6 (at 0 0.5 90) (layer F.SilkS)
-      (effects (font (size 1 1) (thickness 0.15)))
-    )
-    (fp_text value PTT (at 0 -0.5 90) (layer F.Fab)
-      (effects (font (size 1 1) (thickness 0.15)))
-    )
-    (fp_line (start -0.75 2.25) (end 0.75 2.25) (layer F.Fab) (width 0.1))
-    (fp_line (start 0.75 2.25) (end 0.75 6.25) (layer F.Fab) (width 0.1))
-    (fp_line (start 0.75 6.25) (end -1.25 6.25) (layer F.Fab) (width 0.1))
-    (fp_line (start 0.81 4.25) (end 0.81 6.31) (layer F.SilkS) (width 0.12))
-    (fp_line (start -1.31 4.25) (end -1.31 6.31) (layer F.SilkS) (width 0.12))
-    (fp_line (start -1.31 4.25) (end 0.81 4.25) (layer F.SilkS) (width 0.12))
-    (fp_line (start 1.25 1.75) (end -1.75 1.75) (layer F.CrtYd) (width 0.05))
-    (fp_line (start -1.75 1.75) (end -1.75 6.75) (layer F.CrtYd) (width 0.05))
-    (fp_line (start -1.75 6.75) (end 1.25 6.75) (layer F.CrtYd) (width 0.05))
-    (fp_line (start -1.25 6.25) (end -1.25 2.75) (layer F.Fab) (width 0.1))
-    (fp_line (start 1.25 6.75) (end 1.25 1.75) (layer F.CrtYd) (width 0.05))
-    (fp_line (start -1.31 3.25) (end -1.31 2.19) (layer F.SilkS) (width 0.12))
-    (fp_line (start -1.31 2.19) (end -0.25 2.19) (layer F.SilkS) (width 0.12))
-    (fp_line (start -1.25 2.75) (end -0.75 2.25) (layer F.Fab) (width 0.1))
-    (fp_line (start -1.31 6.31) (end 0.81 6.31) (layer F.SilkS) (width 0.12))
-    (fp_text user %R (at -0.25 4.25) (layer F.Fab)
-      (effects (font (size 1 1) (thickness 0.15)))
-    )
-    (pad 2 thru_hole oval (at -0.25 5.25 270) (size 1.35 1.35) (drill 0.8) (layers *.Cu *.Mask)
-      (net 14 "Net-(J6-Pad2)"))
-    (pad 1 thru_hole rect (at -0.25 3.25 270) (size 1.35 1.35) (drill 0.8) (layers *.Cu *.Mask)
-      (net 1 GND))
   )
   (module Capacitor_SMD:CP_Elec_6.3x7.7 (layer F.Cu)
@@
     (polygon
       (pts
-        (xy 246 123) (xy 77 123) (xy 77 44) (xy 246 44)
+        (xy 247.1 123.8) (xy 77 123.8) (xy 77 43.5) (xy 247.1 43.5)
       )
     )
@@
     (polygon
       (pts
-        (xy 246 123) (xy 77 123) (xy 77 44) (xy 246 44)
+        (xy 246.2 123.5) (xy 76.9 123.5) (xy 76.9 43.5) (xy 246.2 43.5)
       )
     )

Commit message: CHANGED BOARD SIZE
Parts:
- moved C3 37.3 mm to (114.1, 67.8), turned to 180 degrees
- moved C2 22.2 mm to (120.9, 70.8)
- moved J3 20.9 mm to (140.7, 112.0)
- moved EC1 18.9 mm to (182.5, 107.7)
- moved VR1 18.4 mm to (117.5, 67.0)
- moved JP1 15.3 mm to (129.5, 97.2)
- moved L1 15.2 mm to (206.5, 104.0), turned to 270 degrees
- moved C1 15.1 mm to (224.0, 77.5)
- moved T2 15.1 mm to (199.9, 97.8)
- moved R3 15.0 mm to (106.7, 82.6)
- moved T1 15.0 mm to (125.5, 69.9)
- moved R5 12.4 mm to (173.7, 103.0)
- moved Q3 11.6 mm to (163.7, 98.0)
- moved C7 11.4 mm to (170.2, 112.5)
- moved R9 11.4 mm to (163.0, 110.3)
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Routing:
- net TRANSMIT_ON: track 57.0 -> 42.3 mm
- net Net-(K1-Pad9): track 44.3 -> 32.6 mm, vias 2 -> 0
- net +12V: track 133.3 -> 123.3 mm, vias 0 -> 2
- net Net-(EC2-Pad1): track 57.7 -> 48.0 mm
- net Net-(C1-Pad1): track 38.3 -> 47.1 mm
- net LPF: track 73.3 -> 66.0 mm
- net /Q2Drain: track 37.4 -> 30.8 mm
- net Net-(J3-Pad1): track 104.9 -> 111.3 mm
- net Net-(C6-Pad2): track 15.7 -> 9.52 mm
- net Net-(C2-Pad1): track 18.5 -> 13.3 mm
- net BIAS: track 38.0 -> 33.1 mm
- net /Q3Drain: track 37.1 -> 32.8 mm
- net Net-(C5-Pad2): track 10.6 -> 6.74 mm
- net Net-(J1-PadS): track 41.7 -> 38.9 mm, vias 0 -> 1
- net Net-(C4-Pad1): track 11.1 -> 8.99 mm
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Other:
- board size 170.9 x 81 mm -> 152.5 x 68.5 mm
