File: 70W-Amplifier.kicad_pcb (KiCad board)
At the start: 2 copper layers, 133.5 x 68 mm, 35 parts, among them J1 RF_OUT, J2 RF_IN, J3 LPF_IN, J4 LPF_OUT, J5 13.8V Input, J6 PTT, K1 G5V-2, Q1 2N3906-SMD, Q2 IRF530, Q3 IRF530, T1 BN-43-202 1T:2T, T2 Ferrite 1T:3T, U1 L7805

Commit message: added dc block cap
Parts:
- added C8: .1uF, Xenir:Capacitor 1206, F.Cu at (202.5, 98.4)
Connections:
- J3 pad 1: Net-(J3-Pad1) -> Net-(C8-Pad1)
- JP1 pad 1: Net-(J3-Pad1) -> Net-(C8-Pad1)
- T2 pad 1: Net-(J3-Pad1) -> Net-(C8-Pad2)
Routing:
- net Net-(J3-Pad1): track 100.0 -> 0.00 mm, vias 2 -> 0
- net Net-(C8-Pad1): track 0.00 -> 94.9 mm, vias 0 -> 2
- net Net-(C8-Pad2): track 0.00 -> 4.32 mm

Commit message: added diode prot
Parts:
- added BIAS_IN1: Conn_01x01, Connector_PinHeader_1.00mm:PinHeader_1x01_P1.00mm_Vertical, F.Cu at (155.5, 70.5)
- added BIAS_OUT1: Conn_01x01, Connector_PinHeader_1.00mm:PinHeader_1x01_P1.00mm_Vertical, F.Cu at (148.5, 70.5)
- added D2: 1N914, Diode_SMD:D_SOD-323, F.Cu at (155.5, 76.5)
- added D3: 1N914, Diode_SMD:D_SOD-323, F.Cu at (148.5, 76.5)
- added D4: 1N914, Diode_SMD:D_SOD-323, F.Cu at (155.5, 81.5)
- added D5: 1N914, Diode_SMD:D_SOD-323, F.Cu at (148.5, 81.5)
- added D6: 1N914, Diode_SMD:D_SOD-323, F.Cu at (155.5, 86.0)
- added D7: 1N914, Diode_SMD:D_SOD-323, F.Cu at (148.5, 86.0)
Routing:
- net Net-(D6-Pad1): track 0.00 -> 9.41 mm
- net Net-(BIAS_OUT1-Pad1): track 0.00 -> 5.00 mm
- net Net-(BIAS_IN1-Pad1): track 0.00 -> 5.00 mm
- net Net-(D3-Pad2): track 0.00 -> 2.85 mm
- net Net-(D2-Pad1): track 0.00 -> 2.80 mm
- net Net-(D5-Pad2): track 0.00 -> 2.40 mm
- net Net-(D4-Pad1): track 0.00 -> 2.40 mm
- net /Q3Drain: track 28.3 -> 30.2 mm
Other:
- outline, holes or cut-outs redrawn

Commit message: fixed diode
Parts:
- removed BIAS_IN1, BIAS_OUT1: Conn_01x01, Connector_PinHeader_1.00mm:PinHeader_1x01_P1.00mm_Vertical
- added J7: Conn_01x02, Xenir:PinPad, F.Cu at (128.5, 56.0)
- added J8: Conn_01x02, Connector_PinHeader_2.54mm:PinHeader_1x02_P2.54mm_Vertical, F.Cu at (151.0, 68.5)
- R7: value 1k -> 180
- moved D3 2.00 mm to (150.5, 76.5)
- moved D5 2.00 mm to (150.5, 81.5)
- moved D7 2.00 mm to (150.5, 86.0)
- moved D2 1.50 mm to (154.0, 76.5)
- moved D4 1.50 mm to (154.0, 81.5)
- moved D6 1.50 mm to (154.0, 86.0)
Routing:
- net Net-(C2-Pad1): track 13.3 -> 27.7 mm
- net Net-(D6-Pad1): track 9.41 -> 5.91 mm
- net Net-(D3-Pad1): track 5.00 -> 7.21 mm
- net Net-(D2-Pad2): track 5.00 -> 7.19 mm

Commit message: changed diode to sod-123
Parts:
- D2, D3, D4, D5, D6, D7: footprint Diode_SMD:D_SOD-323 -> Diode_SMD:D_SOD-123
- moved D6 5.05 mm to (154.0, 91.0)
- moved D7 5.05 mm to (150.5, 91.0)
- moved D4 3.70 mm to (154.0, 85.2)
- moved D5 3.70 mm to (150.5, 85.2)
- moved D3 2.65 mm to (150.5, 79.2)
- moved D2 2.60 mm to (154.0, 79.2)
Routing:
- net Net-(D6-Pad1): track 5.91 -> 3.50 mm
- net Net-(D3-Pad1): track 7.21 -> 9.21 mm
- net Net-(D2-Pad2): track 7.19 -> 9.19 mm

Commit message: Update 70W-Amplifier.kicad_pcb
Other:
- board text added: "From TX"
- board text added: "IN"
- board text added: "LPF BYPASS"
- board text added: "OUT"
- board text added: "PTT"
- board text added: "To ANT"
Changed lines of the file:
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@@
-(kicad_pcb (version 20171130) (host pcbnew 5.1.12-unknown-nightly-202112011503)
+(kicad_pcb (version 20171130) (host pcbnew "(5.1.5)-3")
   (general
     (thickness 1.6)
-    (drawings 28)
+    (drawings 34)
     (tracks 313)
     (zones 0)
@@
   )
   (setup
-    (last_trace_width 0.5)
+    (last_trace_width 0.25)
     (user_trace_width 0.5)
     (user_trace_width 1)
@@
     (tags SOD-123)
     (attr smd)
-    (fp_text reference D7 (at 0 -2 90) (layer F.SilkS)
+    (fp_text reference D7 (at -0.1 1.9 90) (layer F.SilkS)
       (effects (font (size 1 1) (thickness 0.15)))
     )
@@
     (tags SOD-123)
     (attr smd)
-    (fp_text reference D6 (at 0 -2 90) (layer F.SilkS)
+    (fp_text reference D6 (at 0.1 2.1 90) (layer F.SilkS)
       (effects (font (size 1 1) (thickness 0.15)))
     )
@@
     (tags SOD-123)
     (attr smd)
-    (fp_text reference D5 (at 0 -2 90) (layer F.SilkS)
+    (fp_text reference D5 (at 0.05 1.9 90) (layer F.SilkS)
       (effects (font (size 1 1) (thickness 0.15)))
     )
@@
     (tags SOD-123)
     (attr smd)
-    (fp_text reference D4 (at 0 -2 90) (layer F.SilkS)
+    (fp_text reference D4 (at 0 2.2 90) (layer F.SilkS)
       (effects (font (size 1 1) (thickness 0.15)))
     )
@@
     (tags SOD-123)
     (attr smd)
-    (fp_text reference D3 (at 0 -2 90) (layer F.SilkS)
+    (fp_text reference D3 (at -0.05 1.9 90) (layer F.SilkS)
       (effects (font (size 1 1) (thickness 0.15)))
     )
@@
     (tags SOD-123)
     (attr smd)
-    (fp_text reference D2 (at 0 -2 90) (layer F.SilkS)
+    (fp_text reference D2 (at 0.05 2.1 90) (layer F.SilkS)
       (effects (font (size 1 1) (thickness 0.15)))
     )
@@
     (descr http://omronfs.omron.com/en_US/ecb/products/pdf/en-g5v2.pdf)
     (tags "Omron G5V-2 Relay DPDT")
-    (fp_text reference K1 (at 3.81 -2.5) (layer F.SilkS)
+    (fp_text reference K1 (at 3.806 2.78) (layer F.SilkS)
       (effects (font (size 1 1) (thickness 0.15)))
     )
@@
     (descr "Diode, DO-35_SOD27 series, Axial, Horizontal, pin pitch=7.62mm, , length*diameter=4*2mm^2, , http://www.diodes.com/_files/packages/DO-35.pdf")
     (tags "Diode DO-35_SOD27 series Axial Horizontal pin pitch 7.62mm  length 4mm diameter 2mm")
-    (fp_text reference D1 (at 3.81 -2.12) (layer F.SilkS)
+    (fp_text reference D1 (at 4.1 0.1) (layer F.SilkS)
       (effects (font (size 1 1) (thickness 0.15)))
     )
@@
       (net 2 "Net-(C1-Pad1)"))
   )
+  (gr_text "To ANT" (at 83.1 89) (layer F.SilkS)
+    (effects (font (size 1 1) (thickness 0.15)))
+  )
+  (gr_text "From TX" (at 83.1 55.6) (layer F.SilkS)
+    (effects (font (size 1 1) (thickness 0.15)))
+  )
+  (gr_text PTT (at 94.3 85.8) (layer F.SilkS)
+    (effects (font (size 1 1) (thickness 0.15)))
+  )
+  (gr_text "LPF BYPASS" (at 126.2 99) (layer F.SilkS)
+    (effects (font (size 0.5 0.5) (thickness 0.125)))
+  )
+  (gr_text OUT (at 150.7 66) (layer F.SilkS)
+    (effects (font (size 1 1) (thickness 0.15)))
+  )
+  (gr_text IN (at 154 66) (layer F.SilkS)
+    (effects (font (size 1 1) (thickness 0.15)))
+  )
   (gr_line (start 151.5 99) (end 144.5 99) (layer Edge.Cuts) (width 0.1))

Commit message: shrank board
Parts:
- D1: footprint Diode_THT:D_DO-35_SOD27_P7.62mm_Horizontal -> Diode_SMD:D_SOD-123
- moved D1 11.0 mm to (105.5, 75.5)
- moved J6 10.8 mm to (98.1, 83.7)
- moved R2 10.8 mm to (103.2, 87.6)
- moved K1 7.07 mm to (108.9, 71.8)
- moved J1 6.33 mm to (89.5, 95.5)
- moved J2 5.99 mm to (89.6, 64.9)
- moved C3 4.36 mm to (113.8, 63.4), turned to 90 degrees
- moved R3 1.96 mm to (108.6, 82.5)
- moved Q1 1.50 mm to (103.5, 94.0)
- moved R1 1.50 mm to (103.2, 96.6)
Routing:
- net Net-(J2-PadS): track 9.56 -> 5.85 mm
- net Net-(J1-PadS): track 38.9 -> 42.5 mm
- net LPF: track 65.2 -> 68.8 mm
- net BIAS: track 33.1 -> 31.8 mm
- net Net-(K1-Pad9): track 32.6 -> 33.6 mm, vias 0 -> 2
- net TRANSMIT_ON: track 40.2 -> 41.0 mm
- net GND: vias 139 -> 146
Other:
- board size 133.5 x 68 mm -> 127.5 x 68 mm
- board text added: "LPF IN"
- board text added: "LPF OUT"
